File: kicad/iGrillRPiSSRCtl.kicad_pcb (KiCad board)
At the start: 2 copper layers, 7 parts, among them J1 Raspberry_Pi_2_3, J2 Conn_01x02

Commit message: Rev *A changes
Parts:
- D1: value LED -> Low Battery
- D2: value LED -> Done
- J1: moved to B.Cu
- J2: value Conn_01x02 -> SSR Control
- moved R2 54.3 mm to (103.4, 111.8)
- moved BZ1 52.8 mm to (78.0, 109.0), turned to 0 degrees
- moved J2 44.9 mm to (93.7, 111.8), turned to 180 degrees
- moved R1 35.7 mm to (111.0, 108.7), turned to 180 degrees
- moved D2 30.9 mm to (115.3, 111.8), turned to 90 degrees
- moved D1 21.6 mm to (99.1, 111.8), turned to 90 degrees
- moved J1 2.17 mm to (126.2, 103.4), turned to 90 degrees
Connections:
- J1 pad 14: GND -> Net-(J1-Pad14)
- J1 pad 20: GND -> Net-(J1-Pad20)
- J1 pad 25: GND -> Net-(J1-Pad25)
- J1 pad 30: GND -> Net-(J1-Pad30)
- J1 pad 32: Net-(BZ1-Pad2) -> Net-(J1-Pad32)
- J1 pad 33: Net-(J1-Pad33) -> Net-(BZ1-Pad2)
- J1 pad 34: GND -> Net-(J1-Pad34)
- J1 pad 39: GND -> Net-(J1-Pad39)
- J1 pad 6: GND -> Net-(J1-Pad6)
- J1 pad 9: GND -> Net-(J1-Pad9)
- J2 pad 2: Net-(J1-Pad33) -> Net-(J1-Pad32)
- R1 pad 1: Net-(J1-Pad11) -> Net-(J1-Pad16)
- R2 pad 1: Net-(J1-Pad36) -> Net-(J1-Pad15)
Routing:
- net Net-(J1-Pad15): track 0.00 -> 10.5 mm
- net Net-(J1-Pad32): track 0.00 -> 6.58 mm
- net Net-(BZ1-Pad2): track 0.00 -> 6.56 mm
- net Net-(D1-Pad1): track 0.00 -> 5.58 mm
- net Net-(D2-Pad1): track 0.00 -> 4.32 mm
- net Net-(J1-Pad16): track 0.00 -> 3.85 mm
- net +5V: track 0.00 -> 0.72 mm
- added copper zone on B.Cu, net +5V
- added copper zone on F.Cu, net +5V
Other:
- board outline added: 51.8 x 11.7 mm
- rule trace_min: 0.2 -> 0.1524

Commit message: Finishing *A layout
Parts:
- added G***: LOGO, iGrillSmoker:igrill-smoker-url-qr-code, B.Cu at (109.0, 110.2)
- added G***: LOGO, iGrillSmoker:WiFiThem, B.Cu at (123.7, 110.2)
- added G***: LOGO, iGrillSmoker:WiFiThem, F.Cu at (123.7, 110.2)
- moved J2 3.87 mm to (90.2, 110.2), turned to 0 degrees
- moved R2 1.78 mm to (105.2, 111.8)
- moved D1 1.78 mm to (100.8, 111.8)
- moved D2 1.78 mm to (117.1, 111.8)
- moved R1 1.78 mm to (112.8, 108.7)
Routing:
- net Net-(J1-Pad16): track 3.85 -> 5.48 mm
- net Net-(J1-Pad32): track 6.58 -> 7.63 mm
- net Net-(BZ1-Pad2): track 6.56 -> 7.39 mm
- net Net-(J1-Pad15): track 10.5 -> 9.75 mm
Other:
- rule via_min_size: 0.4 -> 0.508
- board text added: "+"
- board text added: "-"
- board text added: "Rev. *A"
- board text added: "Scott Atkins (Scott@kins.dev) https://git.kins.dev/igrill-smoker/"

Commit message: Board update for parts
Parts:
- BZ1: footprint Buzzer_Beeper:Buzzer_12x9.5RM7.6 -> Buzzer_Beeper:Buzzer_TDK_PS1240P02BT_D12.2mm_H6.5mm
- R1, R2: value R -> 100
Changed lines of the file:
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@@
-(kicad_pcb (version 20171130) (host pcbnew "(5.1.2)-2")
+(kicad_pcb (version 20171130) (host pcbnew 5.1.2-f72e74a~84~ubuntu18.04.1)
   (general
     (thickness 1.6)
@@
   )
   (layers
-    (0 F.Cu signal hide)
-    (31 B.Cu signal hide)
-    (32 B.Adhes user hide)
-    (33 F.Adhes user hide)
-    (34 B.Paste user hide)
-    (35 F.Paste user hide)
+    (0 F.Cu signal)
+    (31 B.Cu signal)
+    (32 B.Adhes user)
+    (33 F.Adhes user)
+    (34 B.Paste user)
+    (35 F.Paste user)
     (36 B.SilkS user)
-    (37 F.SilkS user hide)
+    (37 F.SilkS user)
     (38 B.Mask user)
     (39 F.Mask user)
@@
     (add_net "Net-(J1-Pad8)")
     (add_net "Net-(J1-Pad9)")
+  )
+  (module Buzzer_Beeper:Buzzer_TDK_PS1240P02BT_D12.2mm_H6.5mm (layer F.Cu)
+    (at 77.998 108.966)
+    (descr "Buzzer, D12.2mm height 6.5mm, https://product.tdk.com/info/en/catalog/datasheets/piezoelectronic_buzzer_ps_en.pdf")
+    (tags buzzer)
+    (fp_text reference BZ1 (at 3.79 5.08) (layer F.SilkS) hide
+      (effects (font (size 1 1) (thickness 0.15)))
+    )
+    (fp_text value Buzzer (at 3.8 0) (layer F.SilkS)
+      (effects (font (size 1 1) (thickness 0.15)))
+    )
+    (fp_arc (start 2.5 0) (end -3.9 -1.5) (angle -26.38121493) (layer F.SilkS) (width 0.12))
+    (fp_line (start -1.3 -1) (end -1.3 1) (layer F.Fab) (width 0.1))
+    (fp_circle (center 2.5 0) (end 8.73 0) (layer F.SilkS) (width 0.12))
+    (fp_circle (center 2.5 0) (end 3.5 0) (layer F.Fab) (width 0.1))
+    (fp_circle (center 2.5 0) (end 8.6 0) (layer F.Fab) (width 0.1))
+    (fp_circle (center 2.5 0) (end 8.85 0) (layer F.CrtYd) (width 0.05))
+    (fp_text user %R (at 3.8 -4) (layer F.Fab)
+      (effects (font (size 1 1) (thickness 0.15)))
+    )
+    (fp_text user + (at -0.01 -2.54) (layer F.SilkS)
+      (effects (font (size 1 1) (thickness 0.15)))
+    )
+    (pad 2 thru_hole circle (at 5 0) (size 2 2) (drill 1) (layers *.Cu *.Mask)
+      (net 2 "Net-(BZ1-Pad2)"))
+    (pad 1 thru_hole rect (at 0 0) (size 2 2) (drill 1) (layers *.Cu *.Mask)
+      (net 1 +5V))
+    (model ${KISYS3DMOD}/Buzzer_Beeper.3dshapes/Buzzer_TDK_PS1240P02BT_D12.2mm_H6.5mm.wrl
+      (at (xyz 0 0 0))
+      (scale (xyz 1 1 1))
+      (rotate (xyz 0 0 0))
+    )
   )
   (module iGrillSmoker:igrill-smoker-url-qr-code (layer B.Cu)
@@
     )
   )
-  (module Buzzer_Beeper:Buzzer_12x9.5RM7.6 (layer F.Cu)
-    (at 77.998 108.966)
-    (descr "Generic Buzzer, D12mm height 9.5mm with RM7.6mm")
-    (tags buzzer)
-    (fp_text reference BZ1 (at 3.79 5.08) (layer F.SilkS) hide
-      (effects (font (size 1 1) (thickness 0.15)))
-    )
-    (fp_text value Buzzer (at 3.8 0) (layer F.SilkS)
-      (effects (font (size 1 1) (thickness 0.15)))
-    )
-    (fp_text user + (at -0.01 -2.54) (layer F.Fab)
-      (effects (font (size 1 1) (thickness 0.15)))
-    )
-    (fp_text user + (at -0.01 -2.54) (layer F.SilkS)
-      (effects (font (size 1 1) (thickness 0.15)))
-    )
-    (fp_text user %R (at 3.8 -4) (layer F.Fab)
-      (effects (font (size 1 1) (thickness 0.15)))
-    )
-    (fp_circle (center 3.8 0) (end 10.05 0) (layer F.CrtYd) (width 0.05))
-    (fp_circle (center 3.8 0) (end 9.8 0) (layer F.Fab) (width 0.1))
-    (fp_circle (center 3.8 0) (end 4.8 0) (layer F.Fab) (width 0.1))
-    (fp_circle (center 3.8 0) (end 9.9 0) (layer F.SilkS) (width 0.12))
-    (pad 1 thru_hole rect (at 0 0) (size 2 2) (drill 1) (layers *.Cu *.Mask)
-      (net 1 +5V))
-    (pad 2 thru_hole circle (at 7.6 0) (size 2 2) (drill 1) (layers *.Cu *.Mask)
-      (net 2 "Net-(BZ1-Pad2)"))
-    (model ${KISYS3DMOD}/Buzzer_Beeper.3dshapes/Buzzer_12x9.5RM7.6.wrl
-      (at (xyz 0 0 0))
-      (scale (xyz 1 1 1))
-      (rotate (xyz 0 0 0))
-    )
-  )
   (module LED_THT:LED_D5.0mm (layer F.Cu)
     (at 100.838 111.76 90)
@@
       (effects (font (size 1 1) (thickness 0.15)))
     )
-    (fp_text value R (at 3.81 0) (layer F.SilkS)
+    (fp_text value 100 (at 3.81 0) (layer F.SilkS)
       (effects (font (size 1 1) (thickness 0.15)))
     )
@@
       (effects (font (size 1 1) (thickness 0.15)))
     )
-    (fp_text value R (at 3.81 0) (layer F.SilkS)
+    (fp_text value 100 (at 3.81 0) (layer F.SilkS)
       (effects (font (size 1 1) (thickness 0.15)))
     )
@@
   (segment (start 99.568 108.712) (end 99.06 109.22) (width 0.25) (layer F.Cu) (net 1))
   (segment (start 85.598 103.378) (end 85.598 104.178998) (width 0.25) (layer F.Cu) (net 2))
-  (segment (start 84.748001 104.227999) (end 85.598 103.378) (width 0.3048) (layer F.Cu) (net 2))
-  (segment (start 84.395599 104.580401) (end 84.748001 104.227999) (width 0.3048) (layer F.Cu) (net 2))
-  (segment (start 84.395599 107.763599) (end 84.395599 104.580401) (width 0.3048) (layer F.Cu) (net 2))
-  (segment (start 85.598 108.966) (end 84.395599 107.763599) (width 0.3048) (layer F.Cu) (net 2))
+  (segment (start 83.997999 107.966001) (end 82.998 108.966) (width 0.3048) (layer F.Cu) (net 2))
+  (segment (start 84.260401 107.703599) (end 83.997999 107.966001) (width 0.3048) (layer F.Cu) (net 2))
+  (segment (start 84.260401 104.715599) (end 84.260401 107.703599) (width 0.3048) (layer F.Cu) (net 2))
+  (segment (start 85.598 103.378) (end 84.260401 104.715599) (width 0.3048) (layer F.Cu) (net 2))
   (segment (start 102.108 111.76) (end 100.838 111.76) (width 0.3048) (layer F.Cu) (net 3))
   (segment (start 105.156 108.712) (end 102.108 111.76) (width 0.3048) (layer F.Cu) (net 3))
