File: kicad/iGrillRPiSSRCtl-revsB/iGrillRPiSSRCtl-rev-sB.sch (KiCad schematic (older format))
At the start: 12 parts, among them J1 Conn_01x02, P1 Conn_02x20_Odd_Even, SW1 SW_DPDT_x2

Commit message: File naming consistency *C Board
Parts:
- MK1, MK2, MK3, MK4: symbol iGrillRPiSSRCtl-revSB-rescue:Mounting_Hole-Mechanical -> iGrillRPiSSRCtl-rev-sB-rescue:Mounting_Hole-Mechanical
Changed lines of the file:
@@
 EESchema Schematic File Version 4
-LIBS:iGrillRPiSSRCtl-revSB-cache
+LIBS:iGrillRPiSSRCtl-rev-sB-cache
 EELAYER 29 0
 EELAYER END
@@
 ID_SD and ID_SC PINS:\nThese pins are reserved for HAT ID EEPROM.\n\nAt boot time this I2C interface will be\ninterrogated to look for an EEPROM\nthat identifes the attached board and\nallows automagic setup of the GPIOs\n(and optionally, Linux drivers).\n\nDO NOT USE these pins for anything other\nthan attaching an I2C ID EEPROM. Leave\nunconnected if ID EEPROM not required.
 $Comp
-L iGrillRPiSSRCtl-revSB-rescue:Mounting_Hole-Mechanical MK1
+L iGrillRPiSSRCtl-rev-sB-rescue:Mounting_Hole-Mechanical MK1
 U 1 1 5834FB2E
 P 3000 7200
@@
 $EndComp
 $Comp
-L iGrillRPiSSRCtl-revSB-rescue:Mounting_Hole-Mechanical MK3
+L iGrillRPiSSRCtl-rev-sB-rescue:Mounting_Hole-Mechanical MK3
 U 1 1 5834FBEF
 P 3450 7200
@@
 $EndComp
 $Comp
-L iGrillRPiSSRCtl-revSB-rescue:Mounting_Hole-Mechanical MK2
+L iGrillRPiSSRCtl-rev-sB-rescue:Mounting_Hole-Mechanical MK2
 U 1 1 5834FC19
 P 3000 7400
@@
 $EndComp
 $Comp
-L iGrillRPiSSRCtl-revSB-rescue:Mounting_Hole-Mechanical MK4
+L iGrillRPiSSRCtl-rev-sB-rescue:Mounting_Hole-Mechanical MK4
 U 1 1 5834FC4F
 P 3450 7400
