File: kicad/iGrillRPiSSRCtl-revsC/iGrillRPiSSRCtl-rev-sC.kicad_pcb (KiCad board)
At the start: 2 copper layers, 65 x 56 mm, 21 parts, among them J1 Conn_01x02, P1 Conn_02x20_Odd_Even

Commit message: File naming consistency *C Board
Parts:
- BackLogo: renamed from G***; footprint iGrillRPiSSRCtl-revSB:WiFiThem_18x12 -> iGrillRPiSSRCtl-rev-sC:WiFiThem_18x12
- D2: value Cooking Complete -> Smoking Complete
- G*** (x2): footprint iGrillRPiSSRCtl-revSB:qr-code-12x12 -> iGrillRPiSSRCtl-rev-sC:qr-code-12x12
- G***: footprint iGrillRPiSSRCtl-revSB:WiFiThem_18x12 -> iGrillRPiSSRCtl-rev-sC:WiFiThem_18x12
- R1: value 100 -> 68
Connections:
- P1 pad 10: GND -> +5V
- P1 pad 8: +5V -> GND
Other:
- board text added: "+"
- board text added: "-"
- board text added: "Board Created By: Scott Atkins (Scott@kins.dev) https://git.kins.dev/igrill-smoker/ License: Creative Commons BY-NC-SA"
- board text added: "Rev. *C"
- board text removed: "Rev. *B"

Commit message: Board cleanup
Parts:
- moved R1 26.4 mm to (20.0, 50.5), turned to 0 degrees
- moved R2 24.5 mm to (20.0, 47.2), turned to 0 degrees
- moved D2 2.50 mm to (33.8, 52.5), turned to 270 degrees
- moved G*** 0.58 mm to (24.8, 63.2)
Routing:
- net /GPIO2(SDA1): track 2.76 -> 36.8 mm
- net /GPIO3(SCL1): track 2.83 -> 34.9 mm
- net Net-(D1-Pad1): track 29.2 -> 12.0 mm
- net Net-(D2-Pad1): track 24.7 -> 9.84 mm
- net +5V: track 0.00 -> 0.76 mm
Other:
- outline, holes or cut-outs redrawn
- board text added: "iGrill Smoker Solid State Control Board"
- board text removed: "DISPLAY"
- board text removed: "iGrill Smoker SSR Control"
