File: kicad/iGrillRPiSSRCtl-revsC/iGrillRPiSSRCtl-rev-sC.sch (KiCad schematic (older format))
At the start: 12 parts, among them J1 Conn_01x02, P1 Conn_02x20_Odd_Even, SW1 SW_DPDT_x2

Commit message: Electrical Cleanup of Schematic
Parts:
- P1: symbol Connector_Generic:Conn_02x20_Odd_Even -> Connector_RPi:Conn_02x20_Odd_Even
Connections:
- wire segments 79 -> 83
- no-connect marks 14 -> 13
Changed lines of the file:
@@
 $EndComp
 Wire Wire Line
-	3000 1300 3000 1700
+	3000 1300 3000 1400
 Wire Wire Line
 	3000 2700 2900 2700
@@
 Mounting Holes
 $Comp
-L Connector_Generic:Conn_02x20_Odd_Even P1
+L Connector_RPi:Conn_02x20_Odd_Even P1
 U 1 1 59AD464A
 P 2600 2000
@@
 GPIO21(SPI1_SCK)
 Wire Wire Line
-	3100 1100 3100 1150
-Wire Wire Line
 	3000 2700 3000 3150
 Wire Wire Line
 	3000 2500 3000 2700
 Wire Wire Line
-	3000 2000 3000 2500
+	3000 2000 3000 2100
 Wire Wire Line
 	2300 3000 2300 3150
@@
 	2300 2300 2300 3000
 Wire Wire Line
-	3000 1700 3000 2000
+	3000 1700 3000 1800
 NoConn ~ 4050 2400
 NoConn ~ 1150 2400
@@
 	2900 3000 4150 3000
 Connection ~ 4150 2900
-Wire Wire Line
-	4150 2100 4150 2200
-Wire Wire Line
-	2900 2300 4150 2300
-Wire Wire Line
-	2900 2100 4150 2100
-Wire Wire Line
-	2900 2200 4150 2200
-Connection ~ 4150 2200
-Wire Wire Line
-	4150 2200 4150 2300
 $Comp
 L power:+5V #PWR0101
@@
 Wire Wire Line
 	2900 2800 4150 2800
-$Comp
-L power:GND #PWR0102
-U 1 1 5D145865
-P 4150 2300
-F 0 "#PWR0102" H 4150 2050 50  0001 C CNN
-F 1 "GND" H 4150 2150 50  0000 C CNN
-F 2 "" H 4150 2300 50  0000 C CNN
-F 3 "" H 4150 2300 50  0000 C CNN
-	1    4150 2300
-	1    0    0    -1
-$EndComp
-Connection ~ 4150 2300
-Wire Wire Line
-	2900 1900 4150 1900
-Wire Wire Line
-	2900 1400 4150 1400
-Wire Wire Line
-	2900 1800 4150 1800
-Connection ~ 4150 1800
-Wire Wire Line
-	4150 1800 4150 1900
-Wire Wire Line
-	2900 1600 4150 1600
-Wire Wire Line
-	4150 1600 4150 1800
-Wire Wire Line
-	4150 1900 4150 2100
-Connection ~ 4150 1900
-Connection ~ 4150 2100
-Connection ~ 3100 1150
-Wire Wire Line
-	3100 1150 3100 1200
 $Comp
 L Device:R R1
@@
 	550  2700 650  2700
 Connection ~ 550  1250
-Connection ~ 4150 3000
 $Comp
 L Device:Buzzer BZ1
@@
 Wire Wire Line
 	1150 2200 2400 2200
-Wire Wire Line
-	4150 3000 5550 3000
 $Comp
 L Switch:SW_DPDT_x2 SW1
-U 1 1 5D19CE23
-P 4500 2600
-F 0 "SW1" H 4500 2885 50  0000 C CNN
-F 1 "SW_DPDT_x2" H 4500 2794 50  0000 C CNN
-F 2 "Button_Switch_THT:SW_CuK_JS202011CQN_DPDT_Straight" H 4500 2600 50  0001 C CNN
-F 3 "~" H 4500 2600 50  0001 C CNN
-	1    4500 2600
-	1    0    0    -1
+U 2 1 5D19CE23
+P 4500 2700
+F 0 "SW1" H 4500 2985 50  0000 C CNN
+F 1 "SW_DPDT_x2" H 4500 2894 50  0000 C CNN
+F 2 "Button_Switch_THT:SW_CuK_JS202011CQN_DPDT_Straight" H 4500 2700 50  0001 C CNN
+F 3 "~" H 4500 2700 50  0001 C CNN
+	2    4500 2700
+	-1   0    0    -1
 $EndComp
 Wire Wire Line
@@
 	5050 2700 5550 2700
 Wire Wire Line
-	5550 2700 5550 3000
-Wire Wire Line
-	4700 2500 5550 2500
-NoConn ~ 5550 2500
-Wire Wire Line
-	4500 1500 4500 1150
-Wire Wire Line
 	2900 1500 4500 1500
-Wire Wire Line
-	3100 1150 4500 1150
-Wire Wire Line
-	4150 1400 4150 1600
-Connection ~ 4150 1600
+$Comp
+L power:+5V #PWR0102
+U 1 1 5D15CC6F
+P 5550 2700
+F 0 "#PWR0102" H 5550 2550 50  0001 C CNN
+F 1 "+5V" H 5550 2840 50  0000 C CNN
+F 2 "" H 5550 2700 50  0000 C CNN
+F 3 "" H 5550 2700 50  0000 C CNN
+	1    5550 2700
+	1    0    0    -1
+$EndComp
+Wire Wire Line
+	2900 2300 3000 2300
+Connection ~ 3000 2300
+Wire Wire Line
+	3000 2300 3000 2500
+Wire Wire Line
+	3000 2300 4150 2300
+Wire Wire Line
+	2900 2200 3000 2200
+Connection ~ 3000 2200
+Wire Wire Line
+	3000 2200 3000 2300
+Wire Wire Line
+	3000 2200 4150 2200
+Wire Wire Line
+	2900 2100 3000 2100
+Connection ~ 3000 2100
+Wire Wire Line
+	3000 2100 3000 2200
+Wire Wire Line
+	3000 2100 4150 2100
+Wire Wire Line
+	2900 1900 3000 1900
+Connection ~ 3000 1900
+Wire Wire Line
+	3000 1900 3000 2000
+Wire Wire Line
+	3000 1900 4150 1900
+Wire Wire Line
+	2900 1800 3000 1800
+Connection ~ 3000 1800
+Wire Wire Line
+	3000 1800 3000 1900
+Wire Wire Line
+	3000 1800 4150 1800
+Wire Wire Line
+	2900 1600 3000 1600
+Connection ~ 3000 1600
+Wire Wire Line
+	3000 1600 3000 1700
+Wire Wire Line
+	3000 1600 4150 1600
+Wire Wire Line
+	2900 1400 3000 1400
+Connection ~ 3000 1400
+Wire Wire Line
+	3000 1400 3000 1600
+Wire Wire Line
+	3000 1400 4150 1400
+Wire Wire Line
+	3100 1100 3100 1200
+$Comp
+L power:+5V #PWR0104
+U 1 1 5D16B874
+P 4500 1300
+F 0 "#PWR0104" H 4500 1150 50  0001 C CNN
+F 1 "+5V" H 4500 1440 50  0000 C CNN
+F 2 "" H 4500 1300 50  0000 C CNN
+F 3 "" H 4500 1300 50  0000 C CNN
+	1    4500 1300
+	1    0    0    -1
+$EndComp
+Wire Wire Line
+	4500 1500 4500 1300
+Wire Wire Line
+	4150 2800 4300 2800
 $EndSCHEMATC

Commit message: Board updates
Parts:
- added unit 2 of SW1
- D2: value Done -> Smoking Complete
- J1: footprint Connector_Wire:SolderWirePad_1x02_P3.81mm_Drill0.8mm -> TerminalBlock:TerminalBlock_bornier-2_P5.08mm; symbol Connector_Generic:Conn_01x02 -> dk_Terminal-Blocks-Wire-to-Board:1935161
- R1: value 100 -> 100Ω
- R2: value 100 -> 68Ω
- SW1: value SW_DPDT_x2 -> Off On
Connections:
- wire segments 83 -> 93
- no-connect marks 13 -> 12

Commit message: Fixing pinout for RPi PWMs
Parts:
- removed J1: Conn_01x02, TerminalBlock:TerminalBlock_bornier-2_P5.08mm, symbol dk_Terminal-Blocks-Wire-to-Board:1935161
- added J1: Screw_Terminal_01x02, TerminalBlock:TerminalBlock_bornier-2_P5.08mm, symbol Connector:Screw_Terminal_01x02
Connections:
- wire segments 93 -> 90
Changed lines of the file:
@@
 Wire Wire Line
 	4250 2900 4250 3100
-Wire Wire Line
-	4200 2900 4200 4350
-Connection ~ 4200 2900
 $Comp
 L Device:Buzzer BZ1
 U 1 1 5D165E77
-P 5300 5350
-F 0 "BZ1" V 5258 5502 50  0000 L CNN
-F 1 "Buzzer" V 5349 5502 50  0000 L CNN
-F 2 "Buzzer_Beeper:Buzzer_TDK_PS1240P02BT_D12.2mm_H6.5mm" V 5275 5450 50  0001 C CNN
-F 3 "~" V 5275 5450 50  0001 C CNN
-	1    5300 5350
+P 8800 4450
+F 0 "BZ1" V 8758 4602 50  0000 L CNN
+F 1 "Buzzer" V 8849 4602 50  0000 L CNN
+F 2 "Buzzer_Beeper:Buzzer_TDK_PS1240P02BT_D12.2mm_H6.5mm" V 8775 4550 50  0001 C CNN
+F 3 "~" V 8775 4550 50  0001 C CNN
+	1    8800 4450
 	0    1    1    0
 $EndComp
-Wire Wire Line
-	6550 4250 7950 4250
 NoConn ~ 4800 3250
 NoConn ~ 4800 3350
 NoConn ~ 4800 3450
 NoConn ~ 4800 4150
-NoConn ~ 7950 4250
 NoConn ~ 4800 4550
 NoConn ~ 4850 3100
@@
 L Switch:SW_DPDT_x2 SW1
 U 1 1 5D19CE23
-P 4850 5250
-F 0 "SW1" H 4850 5535 50  0000 C CNN
-F 1 "Off    On" H 4850 5444 50  0000 C CNN
-F 2 "Button_Switch_THT:SW_CuK_JS202011CQN_DPDT_Straight" H 4850 5250 50  0001 C CNN
-F 3 "~" H 4850 5250 50  0001 C CNN
-	1    4850 5250
+P 8350 4350
+F 0 "SW1" H 8350 4635 50  0000 C CNN
+F 1 "Off    On" H 8350 4544 50  0000 C CNN
+F 2 "Button_Switch_THT:SW_CuK_JS202011CQN_DPDT_Straight" H 8350 4350 50  0001 C CNN
+F 3 "~" H 8350 4350 50  0001 C CNN
+	1    8350 4350
 	-1   0    0    -1
 $EndComp
 Wire Wire Line
-	5050 5250 5200 5250
-Wire Wire Line
-	5400 5250 5900 5250
+	8550 4350 8700 4350
+Wire Wire Line
+	8900 4350 9400 4350
 Wire Wire Line
 	6550 3150 8150 3150
@@
 L power:+5V #PWR0102
 U 1 1 5D15CC6F
-P 5900 5250
-F 0 "#PWR0102" H 5900 5100 50  0001 C CNN
-F 1 "+5V" H 5900 5390 50  0000 C CNN
-F 2 "" H 5900 5250 50  0000 C CNN
-F 3 "" H 5900 5250 50  0000 C CNN
-	1    5900 5250
+P 9400 4350
+F 0 "#PWR0102" H 9400 4200 50  0001 C CNN
+F 1 "+5V" H 9400 4490 50  0000 C CNN
+F 2 "" H 9400 4350 50  0000 C CNN
+F 3 "" H 9400 4350 50  0000 C CNN
+	1    9400 4350
 	1    0    0    -1
 $EndComp
@@
 	8150 3150 8150 2950
 Wire Wire Line
-	7800 4450 7950 4450
-Wire Wire Line
-	4600 5150 4650 5150
-$Comp
-L power:+5V #PWR0105
-U 1 1 5D1F537C
-P 4450 5300
-F 0 "#PWR0105" H 4450 5150 50  0001 C CNN
-F 1 "+5V" H 4465 5473 50  0000 C CNN
-F 2 "" H 4450 5300 50  0001 C CNN
-F 3 "" H 4450 5300 50  0001 C CNN
-	1    4450 5300
-	1    0    0    -1
-$EndComp
-Wire Wire Line
-	4650 5350 4450 5350
-Wire Wire Line
-	4450 5350 4450 5300
-Wire Wire Line
-	6050 4350 4600 4350
-Wire Wire Line
-	4600 4350 4600 5150
-Wire Wire Line
 	6050 4450 4400 4450
 Wire Wire Line
 	4400 4450 4400 4700
-Wire Wire Line
-	4300 4350 4300 4700
-Wire Wire Line
-	4200 4350 4300 4350
-$Comp
-L dk_Terminal-Blocks-Wire-to-Board:1935161 J1
-U 1 1 5D15A837
-P 4300 4900
-F 0 "J1" V 4200 4950 50  0000 R CNN
-F 1 "Conn_01x02" V 4200 4800 50  0000 R CNN
-F 2 "TerminalBlock:TerminalBlock_bornier-2_P5.08mm" H 4300 4900 50  0001 C CNN
-F 3 "~" H 4300 4900 50  0001 C CNN
-	1    4300 4900
-	1    0    0    -1
-$EndComp
 $Comp
 L Switch:SW_DPDT_x2 SW1
@@
 Wire Wire Line
 	3500 4150 3500 4100
+Wire Wire Line
+	3500 4150 3200 4150
+Wire Wire Line
+	3200 4150 3200 4600
+Wire Wire Line
+	3200 4600 4300 4600
+Connection ~ 3500 4150
+Wire Wire Line
+	4300 4600 4300 4700
+NoConn ~ 4800 4350
+Wire Wire Line
+	4800 4350 6050 4350
+Wire Wire Line
+	7800 4450 8150 4450
+Wire Wire Line
+	6550 4250 8150 4250
+$Comp
+L Connector:Screw_Terminal_01x02 J1
+U 1 1 5D1FC6DA
+P 4300 4900
+F 0 "J1" V 4172 4712 50  0000 R CNN
+F 1 "Screw_Terminal_01x02" V 4263 4712 50  0000 R CNN
+F 2 "TerminalBlock:TerminalBlock_bornier-2_P5.08mm" H 4300 4900 50  0001 C CNN
+F 3 "~" H 4300 4900 50  0001 C CNN
+	1    4300 4900
+	0    -1   1    0
+$EndComp
 $EndSCHEMATC

Commit message: Updated design to fix issues from protoype
Parts:
- added Q1: Q_NPN_CBE, Package_TO_SOT_THT:TO-92L_Inline, symbol Device:Q_NPN_CBE
- added R3: 100Ω, Resistor_THT:R_Axial_DIN0207_L6.3mm_D2.5mm_P10.16mm_Horizontal, symbol Device:R
- added R4: 1kΩ, Resistor_THT:R_Axial_DIN0207_L6.3mm_D2.5mm_P10.16mm_Horizontal, symbol Device:R
- R1: footprint Resistor_THT:R_Axial_DIN0207_L6.3mm_D2.5mm_P7.62mm_Horizontal -> Resistor_THT:R_Axial_DIN0207_L6.3mm_D2.5mm_P10.16mm_Horizontal
- R2: value 68Ω -> 100Ω; footprint Resistor_THT:R_Axial_DIN0207_L6.3mm_D2.5mm_P7.62mm_Horizontal -> Resistor_THT:R_Axial_DIN0207_L6.3mm_D2.5mm_P10.16mm_Horizontal
Connections:
- wire segments 90 -> 101
Changed lines of the file:
@@
 F 0 "R1" V 4650 2850 50  0000 C CNN
 F 1 "100Ω" V 4750 2850 50  0000 C CNN
-F 2 "Resistor_THT:R_Axial_DIN0207_L6.3mm_D2.5mm_P7.62mm_Horizontal" V 4680 2850 50  0001 C CNN
+F 2 "Resistor_THT:R_Axial_DIN0207_L6.3mm_D2.5mm_P10.16mm_Horizontal" V 4680 2850 50  0001 C CNN
 F 3 "~" H 4750 2850 50  0001 C CNN
 	1    4750 2850
@@
 P 4750 2950
 F 0 "R2" V 4850 2950 50  0000 C CNN
-F 1 "68Ω" V 4750 2950 50  0000 C CNN
-F 2 "Resistor_THT:R_Axial_DIN0207_L6.3mm_D2.5mm_P7.62mm_Horizontal" V 4680 2950 50  0001 C CNN
+F 1 "100Ω" V 4750 2950 50  0000 C CNN
+F 2 "Resistor_THT:R_Axial_DIN0207_L6.3mm_D2.5mm_P10.16mm_Horizontal" V 4680 2950 50  0001 C CNN
 F 3 "~" H 4750 2950 50  0001 C CNN
 	1    4750 2950
@@
 L Device:Buzzer BZ1
 U 1 1 5D165E77
-P 8800 4450
-F 0 "BZ1" V 8758 4602 50  0000 L CNN
-F 1 "Buzzer" V 8849 4602 50  0000 L CNN
-F 2 "Buzzer_Beeper:Buzzer_TDK_PS1240P02BT_D12.2mm_H6.5mm" V 8775 4550 50  0001 C CNN
-F 3 "~" V 8775 4550 50  0001 C CNN
-	1    8800 4450
+P 9550 4450
+F 0 "BZ1" V 9508 4602 50  0000 L CNN
+F 1 "Buzzer" V 9599 4602 50  0000 L CNN
+F 2 "Buzzer_Beeper:Buzzer_TDK_PS1240P02BT_D12.2mm_H6.5mm" V 9525 4550 50  0001 C CNN
+F 3 "~" V 9525 4550 50  0001 C CNN
+	1    9550 4450
 	0    1    1    0
 $EndComp
@@
 $EndComp
 Wire Wire Line
-	8550 4350 8700 4350
-Wire Wire Line
-	8900 4350 9400 4350
+	9300 4350 9350 4350
+Wire Wire Line
+	9650 4350 9750 4350
 Wire Wire Line
 	6550 3150 8150 3150
@@
 L power:+5V #PWR0102
 U 1 1 5D15CC6F
-P 9400 4350
-F 0 "#PWR0102" H 9400 4200 50  0001 C CNN
-F 1 "+5V" H 9400 4490 50  0000 C CNN
-F 2 "" H 9400 4350 50  0000 C CNN
-F 3 "" H 9400 4350 50  0000 C CNN
-	1    9400 4350
+P 10150 4350
+F 0 "#PWR0102" H 10150 4200 50  0001 C CNN
+F 1 "+5V" H 10150 4490 50  0000 C CNN
+F 2 "" H 10150 4350 50  0000 C CNN
+F 3 "" H 10150 4350 50  0000 C CNN
+	1    10150 4350
 	1    0    0    -1
 $EndComp
@@
 	0    -1   1    0
 $EndComp
+$Comp
+L Device:R R3
+U 1 1 5D1D8BF1
+P 8750 4350
+F 0 "R3" V 8650 4350 50  0000 C CNN
+F 1 "100Ω" V 8750 4350 50  0000 C CNN
+F 2 "Resistor_THT:R_Axial_DIN0207_L6.3mm_D2.5mm_P10.16mm_Horizontal" V 8680 4350 50  0001 C CNN
+F 3 "~" H 8750 4350 50  0001 C CNN
+	1    8750 4350
+	0    1    1    0
+$EndComp
+$Comp
+L Device:R R4
+U 1 1 5D1D9F32
+P 9500 4150
+F 0 "R4" V 9400 4150 50  0000 C CNN
+F 1 "1kΩ" V 9500 4150 50  0000 C CNN
+F 2 "Resistor_THT:R_Axial_DIN0207_L6.3mm_D2.5mm_P10.16mm_Horizontal" V 9430 4150 50  0001 C CNN
+F 3 "~" H 9500 4150 50  0001 C CNN
+	1    9500 4150
+	0    1    1    0
+$EndComp
+Wire Wire Line
+	8600 4350 8550 4350
+Wire Wire Line
+	9350 4150 9350 4350
+Connection ~ 9350 4350
+Wire Wire Line
+	9350 4350 9450 4350
+Wire Wire Line
+	9650 4150 9750 4150
+Wire Wire Line
+	9750 4150 9750 4350
+Connection ~ 9750 4350
+Wire Wire Line
+	9750 4350 10150 4350
+$Comp
+L power:GND #PWR05
+U 1 1 5D1E7B7B
+P 9300 4950
+F 0 "#PWR05" H 9300 4700 50  0001 C CNN
+F 1 "GND" H 9300 4800 50  0000 C CNN
+F 2 "" H 9300 4950 50  0000 C CNN
+F 3 "" H 9300 4950 50  0000 C CNN
+	1    9300 4950
+	1    0    0    -1
+$EndComp
+$Comp
+L Device:Q_NPN_CBE Q1
+U 1 1 5D1E8600
+P 9200 4650
+F 0 "Q1" H 9391 4696 50  0000 L CNN
+F 1 "Q_NPN_CBE" H 9391 4605 50  0000 L CNN
+F 2 "Package_TO_SOT_THT:TO-92L_Inline" H 9400 4750 50  0001 C CNN
+F 3 "~" H 9200 4650 50  0001 C CNN
+	1    9200 4650
+	1    0    0    -1
+$EndComp
+Wire Wire Line
+	9300 4350 9300 4450
+Wire Wire Line
+	8900 4350 8950 4350
+Wire Wire Line
+	8950 4350 8950 4650
+Wire Wire Line
+	8950 4650 9000 4650
+Wire Wire Line
+	9300 4850 9300 4950
 $EndSCHEMATC

Commit message: Updates from protoype **
Parts:
- added Q2, Q3: Q_PNP_BCE, Package_TO_SOT_THT:TO-92_Inline, symbol Device:Q_PNP_BCE
- Q1: footprint Package_TO_SOT_THT:TO-92L_Inline -> Package_TO_SOT_THT:TO-92_Inline
Connections:
- wire segments 101 -> 109
Changed lines of the file:
@@
 	5950 3150 6050 3150
 Connection ~ 5950 3950
-Wire Wire Line
-	6050 2850 4900 2850
-Wire Wire Line
-	4900 2950 6050 2950
 Text Label 4900 2850 0    50   ~ 0
 GPIO2(SDA1)
@@
 L Device:R R1
 U 1 1 5D14E11D
-P 4750 2850
-F 0 "R1" V 4650 2850 50  0000 C CNN
-F 1 "100Ω" V 4750 2850 50  0000 C CNN
-F 2 "Resistor_THT:R_Axial_DIN0207_L6.3mm_D2.5mm_P10.16mm_Horizontal" V 4680 2850 50  0001 C CNN
-F 3 "~" H 4750 2850 50  0001 C CNN
-	1    4750 2850
+P 3150 2650
+F 0 "R1" V 3250 2650 50  0000 C CNN
+F 1 "100Ω" V 3150 2650 50  0000 C CNN
+F 2 "Resistor_THT:R_Axial_DIN0207_L6.3mm_D2.5mm_P10.16mm_Horizontal" V 3080 2650 50  0001 C CNN
+F 3 "~" H 3150 2650 50  0001 C CNN
+	1    3150 2650
 	0    1    1    0
 $EndComp
@@
 L Device:R R2
 U 1 1 5D14F1BC
-P 4750 2950
-F 0 "R2" V 4850 2950 50  0000 C CNN
-F 1 "100Ω" V 4750 2950 50  0000 C CNN
-F 2 "Resistor_THT:R_Axial_DIN0207_L6.3mm_D2.5mm_P10.16mm_Horizontal" V 4680 2950 50  0001 C CNN
-F 3 "~" H 4750 2950 50  0001 C CNN
-	1    4750 2950
+P 3150 3400
+F 0 "R2" V 3250 3400 50  0000 C CNN
+F 1 "100Ω" V 3150 3400 50  0000 C CNN
+F 2 "Resistor_THT:R_Axial_DIN0207_L6.3mm_D2.5mm_P10.16mm_Horizontal" V 3080 3400 50  0001 C CNN
+F 3 "~" H 3150 3400 50  0001 C CNN
+	1    3150 3400
 	0    1    1    0
 $EndComp
@@
 L Device:LED_ALT D1
 U 1 1 5D14FA39
-P 4400 2700
-F 0 "D1" H 4393 2445 50  0000 C CNN
-F 1 "Low Battery" H 4393 2536 50  0000 C CNN
-F 2 "LED_THT:LED_D5.0mm" H 4400 2700 50  0001 C CNN
-F 3 "~" H 4400 2700 50  0001 C CNN
-	1    4400 2700
+P 3750 2650
+F 0 "D1" H 3743 2395 50  0000 C CNN
+F 1 "Low Battery" H 3743 2486 50  0000 C CNN
+F 2 "LED_THT:LED_D5.0mm" H 3750 2650 50  0001 C CNN
+F 3 "~" H 3750 2650 50  0001 C CNN
+	1    3750 2650
 	-1   0    0    1
 $EndComp
@@
 L Device:LED_ALT D2
 U 1 1 5D150925
-P 4400 3100
-F 0 "D2" H 4393 2845 50  0000 C CNN
-F 1 "Smoking Complete" V 4450 3550 50  0000 C CNN
-F 2 "LED_THT:LED_D5.0mm_Clear" H 4400 3100 50  0001 C CNN
-F 3 "~" H 4400 3100 50  0001 C CNN
-	1    4400 3100
+P 3750 3400
+F 0 "D2" H 3750 3600 50  0000 C CNN
+F 1 "Smoking Complete" H 3750 3500 50  0000 C CNN
+F 2 "LED_THT:LED_D5.0mm_Clear" H 3750 3400 50  0001 C CNN
+F 3 "~" H 3750 3400 50  0001 C CNN
+	1    3750 3400
 	-1   0    0    1
 $EndComp
-Wire Wire Line
-	4250 2700 4250 2900
-Wire Wire Line
-	4600 2950 4600 3100
-Wire Wire Line
-	4600 3100 4550 3100
-Wire Wire Line
-	4550 2700 4600 2700
-Wire Wire Line
-	4600 2700 4600 2850
 $Comp
 L power:+5V #PWR0103
 U 1 1 5D15862C
-P 4200 2500
-F 0 "#PWR0103" H 4200 2350 50  0001 C CNN
-F 1 "+5V" H 4200 2640 50  0000 C CNN
-F 2 "" H 4200 2500 50  0000 C CNN
-F 3 "" H 4200 2500 50  0000 C CNN
-	1    4200 2500
-	1    0    0    -1
-$EndComp
-Wire Wire Line
-	4200 2500 4200 2900
-Wire Wire Line
-	4200 2900 4250 2900
-Connection ~ 4250 2900
-Wire Wire Line
-	4250 2900 4250 3100
+P 2950 2200
+F 0 "#PWR0103" H 2950 2050 50  0001 C CNN
+F 1 "+5V" H 2950 2340 50  0000 C CNN
+F 2 "" H 2950 2200 50  0000 C CNN
+F 3 "" H 2950 2200 50  0000 C CNN
+	1    2950 2200
+	1    0    0    -1
+$EndComp
 $Comp
 L Device:Buzzer BZ1
@@
 Wire Wire Line
 	8150 3150 8150 2950
-Wire Wire Line
-	6050 4450 4400 4450
-Wire Wire Line
-	4400 4450 4400 4700
 $Comp
 L Switch:SW_DPDT_x2 SW1
@@
 	-1   0    0    -1
 $EndComp
-Wire Wire Line
-	4050 4250 6050 4250
 $Comp
 L power:+5V #PWR0106
@@
 Wire Wire Line
 	4300 4600 4300 4700
-NoConn ~ 4800 4350
-Wire Wire Line
-	4800 4350 6050 4350
+NoConn ~ 4800 4450
 Wire Wire Line
 	7800 4450 8150 4450
@@
 F 0 "Q1" H 9391 4696 50  0000 L CNN
 F 1 "Q_NPN_CBE" H 9391 4605 50  0000 L CNN
-F 2 "Package_TO_SOT_THT:TO-92L_Inline" H 9400 4750 50  0001 C CNN
+F 2 "Package_TO_SOT_THT:TO-92_Inline" H 9400 4750 50  0001 C CNN
 F 3 "~" H 9200 4650 50  0001 C CNN
 	1    9200 4650
@@
 Wire Wire Line
 	9300 4850 9300 4950
+$Comp
+L Device:Q_PNP_BCE Q3
+U 1 1 5D1FE4C2
+P 2850 3200
+F 0 "Q3" H 3041 3246 50  0000 L CNN
+F 1 "Q_PNP_BCE" H 3041 3155 50  0000 L CNN
+F 2 "Package_TO_SOT_THT:TO-92_Inline" H 3050 3300 50  0001 C CNN
+F 3 "~" H 2850 3200 50  0001 C CNN
+	1    2850 3200
+	1    0    0    1
+$EndComp
+Wire Wire Line
+	6050 2850 4900 2850
+$Comp
+L power:+5V #PWR0105
+U 1 1 5D241237
+P 2950 2950
+F 0 "#PWR0105" H 2950 2800 50  0001 C CNN
+F 1 "+5V" H 2950 3090 50  0000 C CNN
+F 2 "" H 2950 2950 50  0000 C CNN
+F 3 "" H 2950 2950 50  0000 C CNN
+	1    2950 2950
+	1    0    0    -1
+$EndComp
+$Comp
+L power:GND #PWR0108
+U 1 1 5D25CE00
+P 4350 3500
+F 0 "#PWR0108" H 4350 3250 50  0001 C CNN
+F 1 "GND" H 4350 3350 50  0000 C CNN
+F 2 "" H 4350 3500 50  0000 C CNN
+F 3 "" H 4350 3500 50  0000 C CNN
+	1    4350 3500
+	1    0    0    -1
+$EndComp
+Wire Wire Line
+	3900 3400 4350 3400
+Wire Wire Line
+	4350 3400 4350 3500
+Wire Wire Line
+	3900 2650 4350 2650
+Wire Wire Line
+	4350 2650 4350 3400
+Connection ~ 4350 3400
+Wire Wire Line
+	3300 2650 3600 2650
+Wire Wire Line
+	3300 3400 3600 3400
+Wire Wire Line
+	2950 3400 3000 3400
+Wire Wire Line
+	2950 2950 2950 3000
+Wire Wire Line
+	3000 2650 2950 2650
+Wire Wire Line
+	2950 2200 2950 2250
+$Comp
+L Device:Q_PNP_BCE Q2
+U 1 1 5D285884
+P 2850 2450
+F 0 "Q2" H 3041 2496 50  0000 L CNN
+F 1 "Q_PNP_BCE" H 3041 2405 50  0000 L CNN
+F 2 "Package_TO_SOT_THT:TO-92_Inline" H 3050 2550 50  0001 C CNN
+F 3 "~" H 2850 2450 50  0001 C CNN
+	1    2850 2450
+	1    0    0    1
+$EndComp
+Wire Wire Line
+	2650 2450 2650 1850
+Wire Wire Line
+	2650 1850 4900 1850
+Wire Wire Line
+	4900 1850 4900 2850
+Wire Wire Line
+	2650 3200 2650 3750
+Wire Wire Line
+	2650 3750 4650 3750
+Wire Wire Line
+	4650 3750 4650 2950
+Wire Wire Line
+	4650 2950 6050 2950
+Wire Wire Line
+	4050 4250 6050 4250
+Wire Wire Line
+	4800 4450 6050 4450
+Wire Wire Line
+	6050 4350 4400 4350
+Wire Wire Line
+	4400 4350 4400 4700
 $EndSCHEMATC

Commit message: Updating board design
Parts:
- Q1: value Q_NPN_CBE -> Q_NPN_ECB; footprint Package_TO_SOT_THT:TO-92_Inline -> Package_TO_SOT_THT:TO-92_Inline_Wide; symbol Device:Q_NPN_CBE -> Device:Q_NPN_EBC
- Q2, Q3: value Q_PNP_BCE -> Q_PNP_EBC; footprint Package_TO_SOT_THT:TO-92_Inline -> Package_TO_SOT_THT:TO-92_Inline_Wide; symbol Device:Q_PNP_BCE -> Device:Q_PNP_EBC
Changed lines of the file:
@@
 $EndComp
 $Comp
-L Device:Q_NPN_CBE Q1
+L Device:Q_NPN_EBC Q1
 U 1 1 5D1E8600
 P 9200 4650
 F 0 "Q1" H 9391 4696 50  0000 L CNN
-F 1 "Q_NPN_CBE" H 9391 4605 50  0000 L CNN
-F 2 "Package_TO_SOT_THT:TO-92_Inline" H 9400 4750 50  0001 C CNN
+F 1 "Q_NPN_ECB" H 9391 4605 50  0000 L CNN
+F 2 "Package_TO_SOT_THT:TO-92_Inline_Wide" H 9400 4750 50  0001 C CNN
 F 3 "~" H 9200 4650 50  0001 C CNN
 	1    9200 4650
@@
 	9300 4850 9300 4950
 $Comp
-L Device:Q_PNP_BCE Q3
+L Device:Q_PNP_EBC Q3
 U 1 1 5D1FE4C2
 P 2850 3200
 F 0 "Q3" H 3041 3246 50  0000 L CNN
-F 1 "Q_PNP_BCE" H 3041 3155 50  0000 L CNN
-F 2 "Package_TO_SOT_THT:TO-92_Inline" H 3050 3300 50  0001 C CNN
+F 1 "Q_PNP_EBC" H 3041 3155 50  0000 L CNN
+F 2 "Package_TO_SOT_THT:TO-92_Inline_Wide" H 3050 3300 50  0001 C CNN
 F 3 "~" H 2850 3200 50  0001 C CNN
 	1    2850 3200
@@
 	2950 2200 2950 2250
 $Comp
-L Device:Q_PNP_BCE Q2
+L Device:Q_PNP_EBC Q2
 U 1 1 5D285884
 P 2850 2450
 F 0 "Q2" H 3041 2496 50  0000 L CNN
-F 1 "Q_PNP_BCE" H 3041 2405 50  0000 L CNN
-F 2 "Package_TO_SOT_THT:TO-92_Inline" H 3050 2550 50  0001 C CNN
+F 1 "Q_PNP_EBC" H 3041 2405 50  0000 L CNN
+F 2 "Package_TO_SOT_THT:TO-92_Inline_Wide" H 3050 2550 50  0001 C CNN
 F 3 "~" H 2850 2450 50  0001 C CNN
 	1    2850 2450
