File: kicad/iGrillRPiSSRCtl-revsC/iGrillRPiSSRCtl-rev-sC.sch (KiCad schematic (older format))
At the start: 17 parts, among them J1 Screw_Terminal_01x02, P1 Conn_02x20_Odd_Even, Q1 Q_NPN_ECB, Q2 Q_PNP_EBC, Q3 Q_PNP_EBC, SW1 Off On

Commit message: Cleanup and fixes
Parts:
- removed Q2, Q3: Q_PNP_EBC, Package_TO_SOT_THT:TO-92_Inline_Wide, symbol Device:Q_PNP_EBC
- added Q2, Q3: Q_NPN_ECB, Package_TO_SOT_THT:TO-92_Inline_Wide, symbol Device:Q_NPN_EBC
Connections:
- wire segments 109 -> 112
Changed lines of the file:
@@
 F 3 "~" H 3750 2650 50  0001 C CNN
 	1    3750 2650
-	-1   0    0    1
+	1    0    0    1
 $EndComp
 $Comp
@@
 F 3 "~" H 3750 3400 50  0001 C CNN
 	1    3750 3400
-	-1   0    0    1
-$EndComp
-$Comp
-L power:+5V #PWR0103
-U 1 1 5D15862C
-P 2950 2200
-F 0 "#PWR0103" H 2950 2050 50  0001 C CNN
-F 1 "+5V" H 2950 2340 50  0000 C CNN
-F 2 "" H 2950 2200 50  0000 C CNN
-F 3 "" H 2950 2200 50  0000 C CNN
-	1    2950 2200
-	1    0    0    -1
+	1    0    0    1
 $EndComp
 $Comp
@@
 Wire Wire Line
 	9300 4850 9300 4950
-$Comp
-L Device:Q_PNP_EBC Q3
-U 1 1 5D1FE4C2
-P 2850 3200
-F 0 "Q3" H 3041 3246 50  0000 L CNN
-F 1 "Q_PNP_EBC" H 3041 3155 50  0000 L CNN
-F 2 "Package_TO_SOT_THT:TO-92_Inline_Wide" H 3050 3300 50  0001 C CNN
-F 3 "~" H 2850 3200 50  0001 C CNN
-	1    2850 3200
-	1    0    0    1
-$EndComp
 Wire Wire Line
 	6050 2850 4900 2850
@@
 L power:+5V #PWR0105
 U 1 1 5D241237
-P 2950 2950
-F 0 "#PWR0105" H 2950 2800 50  0001 C CNN
-F 1 "+5V" H 2950 3090 50  0000 C CNN
-F 2 "" H 2950 2950 50  0000 C CNN
-F 3 "" H 2950 2950 50  0000 C CNN
-	1    2950 2950
+P 4350 2600
+F 0 "#PWR0105" H 4350 2450 50  0001 C CNN
+F 1 "+5V" H 4350 2750 50  0000 C CNN
+F 2 "" H 4350 2600 50  0000 C CNN
+F 3 "" H 4350 2600 50  0000 C CNN
+	1    4350 2600
 	1    0    0    -1
 $EndComp
@@
 L power:GND #PWR0108
 U 1 1 5D25CE00
-P 4350 3500
-F 0 "#PWR0108" H 4350 3250 50  0001 C CNN
-F 1 "GND" H 4350 3350 50  0000 C CNN
-F 2 "" H 4350 3500 50  0000 C CNN
-F 3 "" H 4350 3500 50  0000 C CNN
-	1    4350 3500
+P 2950 3850
+F 0 "#PWR0108" H 2950 3600 50  0001 C CNN
+F 1 "GND" H 2950 3700 50  0000 C CNN
+F 2 "" H 2950 3850 50  0000 C CNN
+F 3 "" H 2950 3850 50  0000 C CNN
+	1    2950 3850
 	1    0    0    -1
 $EndComp
@@
 	3900 3400 4350 3400
 Wire Wire Line
-	4350 3400 4350 3500
-Wire Wire Line
 	3900 2650 4350 2650
 Wire Wire Line
 	4350 2650 4350 3400
-Connection ~ 4350 3400
 Wire Wire Line
 	3300 2650 3600 2650
@@
 	3000 2650 2950 2650
 Wire Wire Line
-	2950 2200 2950 2250
-$Comp
-L Device:Q_PNP_EBC Q2
-U 1 1 5D285884
-P 2850 2450
-F 0 "Q2" H 3041 2496 50  0000 L CNN
-F 1 "Q_PNP_EBC" H 3041 2405 50  0000 L CNN
-F 2 "Package_TO_SOT_THT:TO-92_Inline_Wide" H 3050 2550 50  0001 C CNN
-F 3 "~" H 2850 2450 50  0001 C CNN
-	1    2850 2450
-	1    0    0    1
-$EndComp
-Wire Wire Line
-	2650 2450 2650 1850
+	4350 2600 4350 2650
 Wire Wire Line
 	2650 1850 4900 1850
@@
 	4900 1850 4900 2850
 Wire Wire Line
-	2650 3200 2650 3750
-Wire Wire Line
-	2650 3750 4650 3750
-Wire Wire Line
 	4650 3750 4650 2950
 Wire Wire Line
@@
 Wire Wire Line
 	4400 4350 4400 4700
+$Comp
+L Device:Q_NPN_EBC Q2
+U 1 1 5D24A1F1
+P 2850 2850
+F 0 "Q2" H 3041 2896 50  0000 L CNN
+F 1 "Q_NPN_ECB" H 3041 2805 50  0000 L CNN
+F 2 "Package_TO_SOT_THT:TO-92_Inline_Wide" H 3050 2950 50  0001 C CNN
+F 3 "~" H 2850 2850 50  0001 C CNN
+	1    2850 2850
+	1    0    0    -1
+$EndComp
+Connection ~ 4350 2650
+Wire Wire Line
+	2650 1850 2650 2850
+$Comp
+L power:GND #PWR06
+U 1 1 5D25430C
+P 2950 3100
+F 0 "#PWR06" H 2950 2850 50  0001 C CNN
+F 1 "GND" H 2950 2950 50  0000 C CNN
+F 2 "" H 2950 3100 50  0000 C CNN
+F 3 "" H 2950 3100 50  0000 C CNN
+	1    2950 3100
+	1    0    0    -1
+$EndComp
+$Comp
+L Device:Q_NPN_EBC Q3
+U 1 1 5D254764
+P 2850 3600
+F 0 "Q3" H 3041 3646 50  0000 L CNN
+F 1 "Q_NPN_ECB" H 3041 3555 50  0000 L CNN
+F 2 "Package_TO_SOT_THT:TO-92_Inline_Wide" H 3050 3700 50  0001 C CNN
+F 3 "~" H 2850 3600 50  0001 C CNN
+	1    2850 3600
+	1    0    0    -1
+$EndComp
+Wire Wire Line
+	2950 3050 2950 3100
+Wire Wire Line
+	2650 4050 3350 4050
+Wire Wire Line
+	3350 4050 3350 3750
+Wire Wire Line
+	3350 3750 4650 3750
+Wire Wire Line
+	2650 3600 2650 4050
+Wire Wire Line
+	2950 3800 2950 3850
 $EndSCHEMATC
