File: kicad/iGrillRPiSSRCtl-revsC/iGrillRPiSSRCtl-rev-sC.sch (KiCad schematic (older format))
At the start: 17 parts, among them J1 Screw_Terminal_01x02, P1 Conn_02x20_Odd_Even, Q1 Q_NPN_ECB, Q2 Q_NPN_ECB, Q3 Q_NPN_ECB, SW1 Off On

Commit message: Fixing bad merge
Parts:
- D1: footprint LED_SMD:LED_0402_1005Metric -> LED_THT:LED_D5.0mm
- D2: footprint LED_SMD:LED_0402_1005Metric -> LED_THT:LED_D5.0mm_Clear
- Q1: footprint Package_TO_SOT_SMD:SOT-323_SC-70 -> Package_TO_SOT_THT:TO-92_Inline_Wide
- R1, R2, R3: footprint Resistor_SMD:R_0402_1005Metric -> Resistor_THT:R_Axial_DIN0207_L6.3mm_D2.5mm_P10.16mm_Horizontal
- R4: value 1kΩ -> 1000Ω; footprint Resistor_SMD:R_0402_1005Metric -> Resistor_THT:R_Axial_DIN0207_L6.3mm_D2.5mm_P10.16mm_Horizontal
Connections:
- wire segments 109 -> 108
Changed lines of the file:
@@
 Sheet 1 1
 Title "iGrill Smoker SSR Control Board"
-Date "2019-07-08"
+Date "2019-07-09"
 Rev "*C"
 Comp "Redbud Farms"
@@
 F 0 "R1" V 3250 2650 50  0000 C CNN
 F 1 "100Ω" V 3150 2650 50  0000 C CNN
-F 2 "Resistor_SMD:R_0402_1005Metric" V 3080 2650 50  0001 C CNN
+F 2 "Resistor_THT:R_Axial_DIN0207_L6.3mm_D2.5mm_P10.16mm_Horizontal" V 3080 2650 50  0001 C CNN
 F 3 "~" H 3150 2650 50  0001 C CNN
 	1    3150 2650
@@
 F 0 "R2" V 3250 3400 50  0000 C CNN
 F 1 "100Ω" V 3150 3400 50  0000 C CNN
-F 2 "Resistor_SMD:R_0402_1005Metric" V 3080 3400 50  0001 C CNN
+F 2 "Resistor_THT:R_Axial_DIN0207_L6.3mm_D2.5mm_P10.16mm_Horizontal" V 3080 3400 50  0001 C CNN
 F 3 "~" H 3150 3400 50  0001 C CNN
 	1    3150 3400
@@
 F 0 "D1" H 3743 2395 50  0000 C CNN
 F 1 "Low Battery" H 3743 2486 50  0000 C CNN
-F 2 "LED_SMD:LED_0402_1005Metric" H 3750 2650 50  0001 C CNN
+F 2 "LED_THT:LED_D5.0mm" H 3750 2650 50  0001 C CNN
 F 3 "~" H 3750 2650 50  0001 C CNN
 	1    3750 2650
@@
 F 0 "D2" H 3750 3600 50  0000 C CNN
 F 1 "Smoking Complete" H 3750 3500 50  0000 C CNN
-F 2 "LED_SMD:LED_0402_1005Metric" H 3750 3400 50  0001 C CNN
+F 2 "LED_THT:LED_D5.0mm_Clear" H 3750 3400 50  0001 C CNN
 F 3 "~" H 3750 3400 50  0001 C CNN
 	1    3750 3400
@@
 F 0 "R3" V 8650 4350 50  0000 C CNN
 F 1 "100Ω" V 8750 4350 50  0000 C CNN
-F 2 "Resistor_SMD:R_0402_1005Metric" V 8680 4350 50  0001 C CNN
+F 2 "Resistor_THT:R_Axial_DIN0207_L6.3mm_D2.5mm_P10.16mm_Horizontal" V 8680 4350 50  0001 C CNN
 F 3 "~" H 8750 4350 50  0001 C CNN
 	1    8750 4350
@@
 P 9500 4150
 F 0 "R4" V 9400 4150 50  0000 C CNN
-F 1 "1kΩ" V 9500 4150 50  0000 C CNN
-F 2 "Resistor_SMD:R_0402_1005Metric" V 9430 4150 50  0001 C CNN
+F 1 "1000Ω" V 9600 4200 50  0000 C CNN
+F 2 "Resistor_THT:R_Axial_DIN0207_L6.3mm_D2.5mm_P10.16mm_Horizontal" V 9430 4150 50  0001 C CNN
 F 3 "~" H 9500 4150 50  0001 C CNN
 	1    9500 4150
@@
 F 0 "Q1" H 9391 4696 50  0000 L CNN
 F 1 "Q_NPN_ECB" H 9391 4605 50  0000 L CNN
-F 2 "Package_TO_SOT_SMD:SOT-323_SC-70" H 9400 4750 50  0001 C CNN
+F 2 "Package_TO_SOT_THT:TO-92_Inline_Wide" H 9400 4750 50  0001 C CNN
 F 3 "~" H 9200 4650 50  0001 C CNN
 	1    9200 4650
@@
 	2950 3400 3000 3400
 Wire Wire Line
-	2950 2950 2950 3000
-Wire Wire Line
 	3000 2650 2950 2650

Commit message: Updated schematic, pcb for board id
Connections:
- wire segments 108 -> 111
Changed lines of the file:
@@
 	1    0    0    -1
 $EndComp
-Wire Wire Line
-	8150 3150 8150 3050
 $Comp
 L Switch:SW_DPDT_x2 SW1
@@
 Wire Wire Line
 	2950 3800 2950 3850
+Wire Wire Line
+	6650 2950 6650 3050
+Connection ~ 6650 3050
+Wire Wire Line
+	6650 3050 6650 3250
+Wire Wire Line
+	8150 2950 8150 3150
+Wire Wire Line
+	7600 3050 6650 3050
 $EndSCHEMATC
