File: kicad/iGrillRPiSSRCtl-revsC/iGrillRPiSSRCtl-rev-sC.sch (KiCad schematic (older format))
At the start: 17 parts, among them J1 Screw_Terminal_01x02, P1 Conn_02x20_Odd_Even, Q1 Q_NPN_ECB, Q2 Q_NPN_ECB, Q3 Q_NPN_ECB, SW1 Off On

Commit message: Merge Cleanup
Connections:
- wire segments 110 -> 111
Changed lines of the file:
@@
 Wire Wire Line
 	7600 3050 6650 3050
+Wire Wire Line
+	6550 3050 6650 3050
 $EndSCHEMATC
