File: kicad/iGrillRPiSSRCtl-revsD/iGrillRPiSSRCtl-rev-sD.kicad_pcb (KiCad board)
At the start: 2 copper layers, 65 x 56 mm, 27 parts, among them J1 Screw_Terminal_01x02, P1 Conn_02x20_Odd_Even, Q1 Q_NPN_ECB, Q2 Q_PNP_EBC, Q3 Q_PNP_EBC, SW1 Off On

Commit message: Adding *D
Parts:
- G*** (x2): footprint iGrillRPiSSRCtl-rev-sC:qr-code-12x12 -> iGrillRPiSSRCtl-rev-sD:qr-code-12x12
- G*** (x2): footprint iGrillRPiSSRCtl-rev-sC:WiFiThem_18x12 -> iGrillRPiSSRCtl-rev-sD:WiFiThem_18x12
Other:
- board text added: "Rev. *D"
- board text removed: "Rev. *C"
Changed lines of the file:
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@@
     (title "iGrill Smoker SSR Control")
     (date 2019-07-08)
-    (rev *C)
+    (rev *D)
     (company "Redbud Farms")
     (comment 1 https://creativecommons.org/licenses/by-nc-sa/4.0/)
@@
     )
   )
-  (module iGrillRPiSSRCtl-rev-sC:qr-code-12x12 (layer B.Cu)
+  (module iGrillRPiSSRCtl-rev-sD:qr-code-12x12 (layer B.Cu)
     (at 62 55.512 180)
     (fp_text reference G*** (at 0 7.62) (layer B.SilkS) hide
@@
       (xy -4.910667 -2.878666) (xy -4.910667 -2.54) (xy -2.54 -2.54) (xy -2.54 -4.910666)) (layer B.SilkS) (width 0.01))
   )
-  (module iGrillRPiSSRCtl-rev-sC:qr-code-12x12 (layer F.Cu)
+  (module iGrillRPiSSRCtl-rev-sD:qr-code-12x12 (layer F.Cu)
     (at 71.222 63.132)
     (fp_text reference G*** (at 0 -7.62) (layer F.SilkS) hide
@@
     (fp_line (start 28.00096 -0.59944) (end 27.89936 -0.50038) (layer B.Cu) (width 0.381))
   )
-  (module iGrillRPiSSRCtl-rev-sC:WiFiThem_18x12 (layer B.Cu)
+  (module iGrillRPiSSRCtl-rev-sD:WiFiThem_18x12 (layer B.Cu)
     (at 74.27 63.386 180)
     (fp_text reference G*** (at 1.27 -11.43) (layer B.SilkS) hide
@@
       (xy 3.097088 8.995796)) (layer B.Cu) (width 0.01))
   )
-  (module iGrillRPiSSRCtl-rev-sC:WiFiThem_18x12 (layer F.Cu)
+  (module iGrillRPiSSRCtl-rev-sD:WiFiThem_18x12 (layer F.Cu)
     (at 24.74 63.386)
     (fp_text reference G*** (at 1.27 11.43) (layer F.SilkS) hide
@@
     (effects (font (size 1 1) (thickness 0.15)) (justify right mirror))
   )
-  (gr_text "Rev. *C" (at 78.12 54.8) (layer B.Cu)
+  (gr_text "Rev. *D" (at 78.12 54.8) (layer B.Cu)
     (effects (font (size 1 1) (thickness 0.15)) (justify mirror))
   )
-  (gr_text "Rev. *C" (at 21.0316 54.5468) (layer F.Cu)
+  (gr_text "Rev. *D" (at 21.0316 54.5468) (layer F.Cu)
     (effects (font (size 1 1) (thickness 0.15)))
   )

Commit message: *D changes
Parts:
- added D3: Very Low, LED_SMD:LED_0603_1608Metric, F.Cu at (36.8, 50.7)
- added D4: Low, LED_SMD:LED_0603_1608Metric, F.Cu at (32.8, 50.7)
- added D5: On Target, LED_SMD:LED_0603_1608Metric, F.Cu at (28.7, 50.7)
- added D6: High, LED_SMD:LED_0603_1608Metric, F.Cu at (24.7, 50.7)
- added D7: Very High, LED_SMD:LED_0603_1608Metric, F.Cu at (20.7, 50.7)
- added Q4: Q_NPN_ECB, Package_TO_SOT_SMD:SOT-23, F.Cu at (42.6, 25.7)
- added Q5: Q_NPN_ECB, Package_TO_SOT_SMD:SOT-23, F.Cu at (38.5, 25.7)
- added Q6: Q_NPN_ECB, Package_TO_SOT_SMD:SOT-23, F.Cu at (34.3, 25.7)
- added Q7: Q_NPN_ECB, Package_TO_SOT_SMD:SOT-23, F.Cu at (30.2, 25.7)
- added Q8: Q_NPN_ECB, Package_TO_SOT_SMD:SOT-23, F.Cu at (26.1, 25.7)
- added R5: 100Ω, Resistor_SMD:R_1206_3216Metric, F.Cu at (36.1, 46.6)
- added R6: 100Ω, Resistor_SMD:R_1206_3216Metric, F.Cu at (32.1, 46.6)
- added R7: 100Ω, Resistor_SMD:R_1206_3216Metric, F.Cu at (28.0, 46.6)
- added R8: 100Ω, Resistor_SMD:R_1206_3216Metric, F.Cu at (24.0, 46.6)
- added R9: 100Ω, Resistor_SMD:R_1206_3216Metric, F.Cu at (20.0, 46.6)
- D1: footprint LED_THT:LED_D5.0mm -> LED_SMD:LED_0603_1608Metric
- D2: footprint LED_THT:LED_D5.0mm_Clear -> LED_SMD:LED_0603_1608Metric
- G***: footprint iGrillRPiSSRCtl-rev-sD:qr-code-12x12 -> iGrillRPiSSRCtl-rev-sD:qr-code-10x10_inverted
- Q1: footprint Package_TO_SOT_THT:TO-92_Inline_Wide -> Package_TO_SOT_SMD:SOT-23
- Q2, Q3: value Q_PNP_EBC -> Q_NPN_ECB; footprint Package_TO_SOT_THT:TO-92_Inline_Wide -> Package_TO_SOT_SMD:SOT-23
- R1, R2, R3, R4: footprint Resistor_THT:R_Axial_DIN0207_L6.3mm_D2.5mm_P10.16mm_Horizontal -> Resistor_SMD:R_1206_3216Metric
- moved Q2 40.1 mm to (50.9, 25.7), turned to 270 degrees
- moved Q3 32.2 mm to (46.8, 25.7), turned to 270 degrees
- moved Q1 27.7 mm to (66.9, 44.2), turned to 0 degrees
- moved R3 25.5 mm to (67.9, 40.0), turned to 90 degrees
- moved R4 13.5 mm to (73.8, 35.6), turned to 270 degrees
- moved R1 10.8 mm to (33.9, 60.2), turned to 90 degrees
- moved R2 7.97 mm to (33.9, 54.4), turned to 90 degrees
- moved D1 3.38 mm to (35.9, 60.8)
- moved D2 3.21 mm to (35.9, 55.0)
Connections:
- D1 pad 1: GND -> Net-(D1-Pad1)
- D1 pad 2: Net-(D1-Pad2) -> +5V
- D2 pad 1: GND -> Net-(D2-Pad1)
- D2 pad 2: Net-(D2-Pad2) -> +5V
- P1 pad 8: GND -> +5V
- Q2 pad 1: +5V -> GND
- Q2 pad 2: /GPIO2(SDA1) -> /GPIO10(SPI0_MOSI)
- Q3 pad 1: +5V -> GND
- Q3 pad 2: /GPIO3(SCL1) -> /GPIO22(GEN3)
- R1 pad 1: Net-(D1-Pad2) -> Net-(D1-Pad1)
- R2 pad 1: Net-(D2-Pad2) -> Net-(D2-Pad1)
Routing:
- net GND: track 0.00 -> 40.2 mm
- net Net-(Q2-Pad3): track 4.38 -> 39.4 mm
- net /GPIO2(SDA1): track 35.6 -> 3.81 mm
- net /GPIO3(SCL1): track 29.4 -> 2.66 mm
- net Net-(BZ1-Pad2): track 39.5 -> 13.9 mm
- net Net-(Q3-Pad3): track 10.2 -> 33.5 mm
- net Net-(Q4-Pad3): track 0.00 -> 21.3 mm
- net Net-(Q5-Pad3): track 0.00 -> 21.2 mm
- net Net-(Q6-Pad3): track 0.00 -> 21.2 mm
- net Net-(Q7-Pad3): track 0.00 -> 21.1 mm
- net Net-(Q8-Pad3): track 0.00 -> 21.1 mm
- net Net-(R3-Pad2): track 26.8 -> 7.08 mm
- net Net-(D1-Pad2): track 11.4 -> 0.00 mm
- net Net-(D2-Pad2): track 8.36 -> 0.00 mm
- net /GPIO22(GEN3): track 0.00 -> 3.71 mm
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Other:
- board text added: "RPi iGrill Smoker Solid State Relay Control Board"
- board text removed: "B C E"
- board text removed: "E B C"
- board text removed: "NPN"
- board text removed: "PNP"
- board text removed: "iGrill Smoker Solid State Control Board"

Commit message: *D Complete and sent off
Parts:
- removed R3: 100Ω, Resistor_SMD:R_1206_3216Metric
- added Q9: Q_NPN_ECB, Package_TO_SOT_SMD:SOT-23, F.Cu at (73.4, 26.2)
- BZ1: footprint Buzzer_Beeper:Buzzer_TDK_PS1240P02BT_D12.2mm_H6.5mm -> iGrillRPiSSRCtl-rev-sD:Buzzer_KELIKING_KLJ-1230-smd
- D3: value Very Low -> Hot
- D4: value Low -> Warm
- D5: value On Target -> Perfect
- D6: value High -> Cool
- D7: value Very High -> Cold
- R1, R5, R6, R8, R9: value 100Ω -> 120Ω; footprint Resistor_SMD:R_1206_3216Metric -> Resistor_SMD:R_0603_1608Metric
- R2, R7: value 100Ω -> 82Ω; footprint Resistor_SMD:R_1206_3216Metric -> Resistor_SMD:R_0603_1608Metric
- R4: footprint Resistor_SMD:R_1206_3216Metric -> Resistor_SMD:R_0603_1608Metric
- SW1: value Off On -> Off On; footprint Button_Switch_THT:SW_CuK_JS202011CQN_DPDT_Straight -> iGrillRPiSSRCtl-rev-sD:SW_OS202011MS2QS1
- moved SW1 3.23 mm to (68.9, 32.8)
- moved BZ1 2.75 mm to (75.3, 44.1)
- moved R1 0.66 mm to (33.9, 60.9)
- moved R2 0.61 mm to (33.9, 55.0)
- moved R5 0.51 mm to (36.1, 46.1)
- moved R6 0.51 mm to (32.1, 46.1)
- moved R7 0.51 mm to (28.0, 46.1)
- moved R8 0.51 mm to (24.0, 46.1)
- moved R9 0.51 mm to (20.0, 46.1)
Connections:
- J1 pad 2: /GPIO13(PWM1) -> Net-(J1-Pad2)
- SW1 pad 2: Net-(R3-Pad2) -> Net-(Q1-Pad2)
Routing:
- net Net-(Q1-Pad2): track 4.60 -> 16.2 mm
- net /GPIO13(PWM1): track 15.5 -> 8.14 mm
- net Net-(R3-Pad2): track 7.08 -> 0.00 mm
- net Net-(J1-Pad2): track 0.00 -> 5.75 mm
- net +5V: track 0.00 -> 5.04 mm
- net Net-(Q2-Pad3): track 39.4 -> 43.2 mm
- net Net-(D4-Pad1): track 2.70 -> 6.39 mm
- net Net-(D3-Pad1): track 2.70 -> 6.39 mm
- net Net-(D7-Pad1): track 2.70 -> 6.39 mm
- net Net-(D5-Pad1): track 2.70 -> 5.72 mm
- net Net-(D6-Pad1): track 2.70 -> 5.54 mm
- net /GPIO6: track 13.7 -> 11.9 mm
- net Net-(Q3-Pad3): track 33.5 -> 34.8 mm
- net /GPIO12(PWM0): track 13.3 -> 14.5 mm
- net Net-(BZ1-Pad2): track 13.9 -> 13.1 mm
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Other:
- board text added: "02 - Cold 03 - Cool 04 - Perfect 17 - Warm 22 - Hot 10 - Low Battery 22 - Smoking Complete 06 - Switch 12 - Buzzer 13 - SSR (J1)"
- board text added: "Buzzer Control"
- board text removed: "02 - Red LED 03 - Green LED 06 - Switch 12 - Buzzer 13 - SSR (J1)"
- board text removed: "Buzzer"
