File: kicad/iGrillRPiSSRCtl-revsD/iGrillRPiSSRCtl-rev-sD.sch (KiCad schematic (older format))
At the start: 17 parts, among them J1 Screw_Terminal_01x02, P1 Conn_02x20_Odd_Even, Q1 Q_NPN_ECB, Q2 Q_PNP_EBC, Q3 Q_PNP_EBC, SW1 Off On

Commit message: Adding *D
Parts:
- MK1, MK2, MK3, MK4: symbol iGrillRPiSSRCtl-rev-sC-rescue:Mounting_Hole-Mechanical -> iGrillRPiSSRCtl-rev-sD-rescue:Mounting_Hole-Mechanical
Changed lines of the file:
@@
 EESchema Schematic File Version 4
-LIBS:iGrillRPiSSRCtl-rev-sC-cache
+LIBS:iGrillRPiSSRCtl-rev-sD-cache
 EELAYER 29 0
 EELAYER END
@@
 Title "iGrill Smoker SSR Control Board"
 Date "2019-07-08"
-Rev "*C"
+Rev "*D"
 Comp "Redbud Farms"
 Comment1 "https://creativecommons.org/licenses/by-nc-sa/4.0/"
@@
 ID_SD and ID_SC PINS:\nThese pins are reserved for HAT ID EEPROM.\n\nAt boot time this I2C interface will be\ninterrogated to look for an EEPROM\nthat identifes the attached board and\nallows automagic setup of the GPIOs\n(and optionally, Linux drivers).\n\nDO NOT USE these pins for anything other\nthan attaching an I2C ID EEPROM. Leave\nunconnected if ID EEPROM not required.
 $Comp
-L iGrillRPiSSRCtl-rev-sC-rescue:Mounting_Hole-Mechanical MK1
+L iGrillRPiSSRCtl-rev-sD-rescue:Mounting_Hole-Mechanical MK1
 U 1 1 5834FB2E
 P 3000 7200
@@
 $EndComp
 $Comp
-L iGrillRPiSSRCtl-rev-sC-rescue:Mounting_Hole-Mechanical MK3
+L iGrillRPiSSRCtl-rev-sD-rescue:Mounting_Hole-Mechanical MK3
 U 1 1 5834FBEF
 P 3450 7200
@@
 $EndComp
 $Comp
-L iGrillRPiSSRCtl-rev-sC-rescue:Mounting_Hole-Mechanical MK2
+L iGrillRPiSSRCtl-rev-sD-rescue:Mounting_Hole-Mechanical MK2
 U 1 1 5834FC19
 P 3000 7400
@@
 $EndComp
 $Comp
-L iGrillRPiSSRCtl-rev-sC-rescue:Mounting_Hole-Mechanical MK4
+L iGrillRPiSSRCtl-rev-sD-rescue:Mounting_Hole-Mechanical MK4
 U 1 1 5834FC4F
 P 3450 7400

Commit message: *D changes
Parts:
- removed Q2, Q3: Q_PNP_EBC, Package_TO_SOT_THT:TO-92_Inline_Wide, symbol Device:Q_PNP_EBC
- added D3: Very Low, LED_SMD:LED_0603_1608Metric, symbol Device:LED_ALT
- added D4: Low, LED_SMD:LED_0603_1608Metric, symbol Device:LED_ALT
- added D5: On Target, LED_SMD:LED_0603_1608Metric, symbol Device:LED_ALT
- added D6: High, LED_SMD:LED_0603_1608Metric, symbol Device:LED_ALT
- added D7: Very High, LED_SMD:LED_0603_1608Metric, symbol Device:LED_ALT
- added Q2, Q3, Q4, Q5, Q6, Q7, Q8: Q_NPN_ECB, Package_TO_SOT_SMD:SOT-23, symbol Device:Q_NPN_EBC
- added R5, R6, R7, R8, R9: 100Ω, Resistor_SMD:R_1206_3216Metric, symbol Device:R
- BZ1: Partnumber (none) -> PS1240P02BT
- D1: footprint LED_THT:LED_D5.0mm -> LED_SMD:LED_0603_1608Metric; Partnumber (none) -> 150060RS75000
- D2: footprint LED_THT:LED_D5.0mm_Clear -> LED_SMD:LED_0603_1608Metric; Partnumber (none) -> 150060VS75000
- J1: Partnumber (none) -> TB002-500-02BE
- MK1, MK2, MK3, MK4: Partnumber (none) -> NONE
- P1: Partnumber (none) -> SFH11-PBPC-D20-ST-BK
- Q1: footprint Package_TO_SOT_THT:TO-92_Inline_Wide -> Package_TO_SOT_SMD:SOT-23; Partnumber (none) -> DMN65D8L-7
- R1, R2, R3: footprint Resistor_THT:R_Axial_DIN0207_L6.3mm_D2.5mm_P10.16mm_Horizontal -> Resistor_SMD:R_1206_3216Metric; Partnumber (none) -> RMCF1206JT100R
- R4: footprint Resistor_THT:R_Axial_DIN0207_L6.3mm_D2.5mm_P10.16mm_Horizontal -> Resistor_SMD:R_1206_3216Metric; Partnumber (none) -> RMCF1206JT1K00
- SW1: Partnumber (none) -> JS202011CQN
Connections:
- wire segments 109 -> 136
- no-connect marks 12 -> 7

Commit message: *D Complete and sent off
Parts:
- removed R3: 100Ω, Resistor_SMD:R_1206_3216Metric, symbol Device:R
- added Q9: Q_NPN_ECB, Package_TO_SOT_SMD:SOT-23, symbol Device:Q_NPN_EBC
- BZ1: footprint Buzzer_Beeper:Buzzer_TDK_PS1240P02BT_D12.2mm_H6.5mm -> iGrillRPiSSRCtl-rev-sD:Buzzer_KELIKING_KLJ-1230-smd; Partnumber PS1240P02BT -> KLJ-1230
- D1: Partnumber 150060RS75000 -> 19-217-R6C-AL1M2VY-3T
- D2: Partnumber 150060VS75000 -> 19-217-G7C-AN1P2-3T
- D3: value Very Low -> Hot; Partnumber 150060RS75000 -> 19-217-R6C-AL1M2VY-3T
- D4: value Low -> Warm; Partnumber 150060YS75000 -> 19-217-Y5C-AM1N1VY-3T
- D5: value On Target -> Perfect; Partnumber 150060VS75000 -> 19-217-G7C-AN1P2-3T
- D6: value High -> Cool; Partnumber 150060YS75000 -> 19-217-Y5C-AM1N1VY-3T
- D7: value Very High -> Cold; Partnumber 150060RS75000 -> 19-217-R6C-AL1M2VY-3T
- J1: Partnumber TB002-500-02BE -> 1715721
- MK1, MK2, MK3, MK4: Partnumber NONE -> (none)
- P1: Partnumber SFH11-PBPC-D20-ST-BK -> PF1-M220-SBB-G0-TR
- Q1, Q2, Q3, Q4, Q5, Q6, Q7, Q8: Partnumber DMN65D8L-7 -> MMBT3904LT1G
- R1, R5, R6, R8, R9: value 100Ω -> 120Ω; footprint Resistor_SMD:R_1206_3216Metric -> Resistor_SMD:R_0603_1608Metric; Partnumber RMCF1206JT100R -> RC0603JR-07120RL
- R2, R7: value 100Ω -> 82Ω; footprint Resistor_SMD:R_1206_3216Metric -> Resistor_SMD:R_0603_1608Metric; Partnumber RMCF1206JT100R -> RC0603JR-0782RL
- R4: footprint Resistor_SMD:R_1206_3216Metric -> Resistor_SMD:R_0603_1608Metric; Partnumber RMCF1206JT1K00 -> RC0603JR-075K1L
- SW1: footprint Button_Switch_THT:SW_CuK_JS202011CQN_DPDT_Straight -> iGrillRPiSSRCtl-rev-sD:SW_OS202011MS2QS1; Partnumber JS202011CQN -> JS202011SCQN
Connections:
- wire segments 136 -> 137
