File: kicad/iGrillRPiSSRCtl-revsE/iGrillRPiSSRCtl-rev-sE.sch (KiCad schematic (older format))
At the start: 37 parts, among them J1 Screw_Terminal_01x02, P1 Conn_02x20_Odd_Even, Q1 Q_NPN_ECB, Q2 Q_NPN_ECB, Q3 Q_NPN_ECB, Q4 Q_NPN_ECB, Q5 Q_NPN_ECB, Q6 Q_NPN_ECB, Q7 Q_NPN_ECB, Q8 Q_NPN_ECB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

Commit message: Updating buzzer and design for *e
Parts:
- removed Q1, Q2, Q3, Q4, Q5, Q6, Q7, Q8, Q9: Q_NPN_ECB, Package_TO_SOT_SMD:SOT-23, symbol Device:Q_NPN_EBC
- added Q1, Q2, Q3, Q4, Q5, Q6, Q7, Q8, Q9: MMBT3904LT1G, Package_TO_SOT_SMD:SOT-23, symbol dk_Transistors-Bipolar-BJT-Single:MMBT3904LT1G
- added R10, R11, R13, R15, R16, R2, R4, R6, R8: 180Ω, Resistor_SMD:R_0603_1608Metric, symbol Device:R
- R1, R5: value 120Ω -> 180Ω
- R12: renamed from R8; value 120Ω -> 180Ω
- R14: renamed from R9; value 120Ω -> 180Ω
- R3: renamed from R2; value 82Ω -> 180Ω
- R7: renamed from R6; value 120Ω -> 180Ω
- R9: renamed from R7; value 82Ω -> 180Ω
- renumbered R4 to R17
Connections:
- wire segments 173 -> 179

Commit message: Board Updates
Parts:
- D1: Partnumber 19-217-R6C-AL1M2VY-3T -> Red LED
- D2, D5: Partnumber 19-217-G7C-AN1P2-3T -> Green LED
- D3: value Hot -> Cold; Partnumber 19-217-R6C-AL1M2VY-3T -> Red LED
- D4: value Warm -> Cool; Partnumber 19-217-Y5C-AM1N1VY-3T -> Yellow LED
- D6: value Cool -> Warm; Partnumber 19-217-Y5C-AM1N1VY-3T -> Yellow LED
- D7: value Cold -> Hot; Partnumber 19-217-R6C-AL1M2VY-3T -> Red LED
- J1: Partnumber 1715721 -> Screw Terminal
- P1: Partnumber PF1-M220-SBB-G0-TR -> 40 pin femal connector rectangular
- R1, R10, R11, R12, R13, R14, R15, R16, R2, R4, R5, R6, R7, R8: Partnumber RC0603JR-07120RL -> 180 ohm resistor
- R17: Partnumber RC0603JR-075K1L -> 1k ohm resistor
- R3, R9: Partnumber RC0603JR-0782RL -> 180 ohm resistor
Changed lines of the file:
@@
 Sheet 1 1
 Title "iGrill Smoker SSR Control Board"
-Date "2019-08-01"
+Date "2019-08-02"
 Rev "*E"
 Comp "Redbud Farms"
@@
 F 2 "Connector_PinSocket_2.54mm:PinSocket_2x20_P2.54mm_Vertical" H 1400 2700 50  0001 C CNN
 F 3 "" H 1400 2700 50  0001 C CNN
-F 4 "PF1-M220-SBB-G0-TR" H 6250 3650 50  0001 C CNN "Partnumber"
+F 4 "40 pin femal connector rectangular" H 6250 3650 50  0001 C CNN "Partnumber"
 	1    6250 3650
 	1    0    0    -1
@@
 F 2 "Resistor_SMD:R_0603_1608Metric" V 780 1550 50  0001 C CNN
 F 3 "~" H 850 1550 50  0001 C CNN
-F 4 "RC0603JR-07120RL" H 850 1550 50  0001 C CNN "Partnumber"
+F 4 "180 ohm resistor" H 850 1550 50  0001 C CNN "Partnumber"
 	1    850  1550
 	1    0    0    -1
@@
 F 2 "Resistor_SMD:R_0603_1608Metric" V 1530 1550 50  0001 C CNN
 F 3 "~" H 1600 1550 50  0001 C CNN
-F 4 "RC0603JR-0782RL" H 1600 1550 50  0001 C CNN "Partnumber"
+F 4 "180 ohm resistor" H 1600 1550 50  0001 C CNN "Partnumber"
 	1    1600 1550
 	1    0    0    -1
@@
 F 2 "LED_SMD:LED_0603_1608Metric" H 850 950 50  0001 C CNN
 F 3 "~" H 850 950 50  0001 C CNN
-F 4 "19-217-R6C-AL1M2VY-3T" H 850 950 50  0001 C CNN "Partnumber"
+F 4 "Red LED" H 850 950 50  0001 C CNN "Partnumber"
 	1    850  950
 	0    1    -1   0
@@
 F 2 "LED_SMD:LED_0603_1608Metric" H 1600 950 50  0001 C CNN
 F 3 "~" H 1600 950 50  0001 C CNN
-F 4 "19-217-G7C-AN1P2-3T" H 1600 950 50  0001 C CNN "Partnumber"
+F 4 "Green LED" H 1600 950 50  0001 C CNN "Partnumber"
 	1    1600 950
 	0    1    -1   0
@@
 F 2 "TerminalBlock:TerminalBlock_bornier-2_P5.08mm" H 3650 5150 50  0001 C CNN
 F 3 "~" H 3650 5150 50  0001 C CNN
-F 4 "1715721" H 3650 5150 50  0001 C CNN "Partnumber"
+F 4 "Screw Terminal" H 3650 5150 50  0001 C CNN "Partnumber"
 	1    3650 5150
 	0    -1   1    0
@@
 F 2 "Resistor_SMD:R_0603_1608Metric" V 9430 4150 50  0001 C CNN
 F 3 "~" H 9500 4150 50  0001 C CNN
-F 4 "RC0603JR-075K1L" H 9500 4150 50  0001 C CNN "Partnumber"
+F 4 "1k ohm resistor" H 9500 4150 50  0001 C CNN "Partnumber"
 	1    9500 4150
 	0    1    1    0
@@
 F 2 "Resistor_SMD:R_0603_1608Metric" V 2280 1550 50  0001 C CNN
 F 3 "~" H 2350 1550 50  0001 C CNN
-F 4 "RC0603JR-07120RL" H 2350 1550 50  0001 C CNN "Partnumber"
+F 4 "180 ohm resistor" H 2350 1550 50  0001 C CNN "Partnumber"
 	1    2350 1550
 	1    0    0    -1
@@
 P 2350 950
 F 0 "D3" H 2300 1050 50  0000 C CNN
-F 1 "Hot" H 2150 800 50  0000 C CNN
+F 1 "Cold" H 2150 800 50  0000 C CNN
 F 2 "LED_SMD:LED_0603_1608Metric" H 2350 950 50  0001 C CNN
 F 3 "~" H 2350 950 50  0001 C CNN
-F 4 "19-217-R6C-AL1M2VY-3T" H 2350 950 50  0001 C CNN "Partnumber"
+F 4 "Red LED" H 2350 950 50  0001 C CNN "Partnumber"
 	1    2350 950
 	0    1    -1   0
@@
 F 2 "Resistor_SMD:R_0603_1608Metric" V 3030 1550 50  0001 C CNN
 F 3 "~" H 3100 1550 50  0001 C CNN
-F 4 "RC0603JR-07120RL" H 3100 1550 50  0001 C CNN "Partnumber"
+F 4 "180 ohm resistor" H 3100 1550 50  0001 C CNN "Partnumber"
 	1    3100 1550
 	1    0    0    -1
@@
 P 3100 950
 F 0 "D4" H 3050 1050 50  0000 C CNN
-F 1 "Warm" H 2900 800 50  0000 C CNN
+F 1 "Cool" H 2900 800 50  0000 C CNN
 F 2 "LED_SMD:LED_0603_1608Metric" H 3100 950 50  0001 C CNN
 F 3 "~" H 3100 950 50  0001 C CNN
-F 4 "19-217-Y5C-AM1N1VY-3T" H 3100 950 50  0001 C CNN "Partnumber"
+F 4 "Yellow LED" H 3100 950 50  0001 C CNN "Partnumber"
 	1    3100 950
 	0    1    -1   0
@@
 F 2 "Resistor_SMD:R_0603_1608Metric" V 3780 1550 50  0001 C CNN
 F 3 "~" H 3850 1550 50  0001 C CNN
-F 4 "RC0603JR-0782RL" H 3850 1550 50  0001 C CNN "Partnumber"
+F 4 "180 ohm resistor" H 3850 1550 50  0001 C CNN "Partnumber"
 	1    3850 1550
 	1    0    0    -1
@@
 F 2 "LED_SMD:LED_0603_1608Metric" H 3850 950 50  0001 C CNN
 F 3 "~" H 3850 950 50  0001 C CNN
-F 4 "19-217-G7C-AN1P2-3T" H 3850 950 50  0001 C CNN "Partnumber"
+F 4 "Green LED" H 3850 950 50  0001 C CNN "Partnumber"
 	1    3850 950
 	0    1    -1   0
@@
 F 2 "Resistor_SMD:R_0603_1608Metric" V 4530 1550 50  0001 C CNN
 F 3 "~" H 4600 1550 50  0001 C CNN
-F 4 "RC0603JR-07120RL" H 4600 1550 50  0001 C CNN "Partnumber"
+F 4 "180 ohm resistor" H 4600 1550 50  0001 C CNN "Partnumber"
 	1    4600 1550
 	1    0    0    -1
@@
 P 4600 950
 F 0 "D6" H 4550 1050 50  0000 C CNN
-F 1 "Cool" H 4400 800 50  0000 C CNN
+F 1 "Warm" H 4400 800 50  0000 C CNN
 F 2 "LED_SMD:LED_0603_1608Metric" H 4600 950 50  0001 C CNN
 F 3 "~" H 4600 950 50  0001 C CNN
-F 4 "19-217-Y5C-AM1N1VY-3T" H 4600 950 50  0001 C CNN "Partnumber"
+F 4 "Yellow LED" H 4600 950 50  0001 C CNN "Partnumber"
 	1    4600 950
 	0    1    -1   0
@@
 F 2 "Resistor_SMD:R_0603_1608Metric" V 5280 1550 50  0001 C CNN
 F 3 "~" H 5350 1550 50  0001 C CNN
-F 4 "RC0603JR-07120RL" H 5350 1550 50  0001 C CNN "Partnumber"
+F 4 "180 ohm resistor" H 5350 1550 50  0001 C CNN "Partnumber"
 	1    5350 1550
 	1    0    0    -1
@@
 P 5350 950
 F 0 "D7" H 5300 1050 50  0000 C CNN
-F 1 "Cold" H 5150 800 50  0000 C CNN
+F 1 "Hot" H 5150 800 50  0000 C CNN
 F 2 "LED_SMD:LED_0603_1608Metric" H 5350 950 50  0001 C CNN
 F 3 "~" H 5350 950 50  0001 C CNN
-F 4 "19-217-R6C-AL1M2VY-3T" H 5350 950 50  0001 C CNN "Partnumber"
+F 4 "Red LED" H 5350 950 50  0001 C CNN "Partnumber"
 	1    5350 950
 	0    1    -1   0
@@
 F 2 "Resistor_SMD:R_0603_1608Metric" V 980 2550 50  0001 C CNN
 F 3 "~" H 1050 2550 50  0001 C CNN
-F 4 "RC0603JR-07120RL" H 1050 2550 50  0001 C CNN "Partnumber"
+F 4 "180 ohm resistor" H 1050 2550 50  0001 C CNN "Partnumber"
 	1    1050 2550
 	1    0    0    -1
@@
 F 2 "Resistor_SMD:R_0603_1608Metric" V 1730 2550 50  0001 C CNN
 F 3 "~" H 1800 2550 50  0001 C CNN
-F 4 "RC0603JR-07120RL" H 1800 2550 50  0001 C CNN "Partnumber"
+F 4 "180 ohm resistor" H 1800 2550 50  0001 C CNN "Partnumber"
 	1    1800 2550
 	1    0    0    -1
@@
 F 2 "Resistor_SMD:R_0603_1608Metric" V 2480 2550 50  0001 C CNN
 F 3 "~" H 2550 2550 50  0001 C CNN
-F 4 "RC0603JR-07120RL" H 2550 2550 50  0001 C CNN "Partnumber"
+F 4 "180 ohm resistor" H 2550 2550 50  0001 C CNN "Partnumber"
 	1    2550 2550
 	1    0    0    -1
@@
 F 2 "Resistor_SMD:R_0603_1608Metric" V 3230 2550 50  0001 C CNN
 F 3 "~" H 3300 2550 50  0001 C CNN
-F 4 "RC0603JR-07120RL" H 3300 2550 50  0001 C CNN "Partnumber"
+F 4 "180 ohm resistor" H 3300 2550 50  0001 C CNN "Partnumber"
 	1    3300 2550
 	1    0    0    -1
@@
 F 2 "Resistor_SMD:R_0603_1608Metric" V 3980 2550 50  0001 C CNN
 F 3 "~" H 4050 2550 50  0001 C CNN
-F 4 "RC0603JR-07120RL" H 4050 2550 50  0001 C CNN "Partnumber"
+F 4 "180 ohm resistor" H 4050 2550 50  0001 C CNN "Partnumber"
 	1    4050 2550
 	1    0    0    -1
@@
 F 2 "Resistor_SMD:R_0603_1608Metric" V 4730 2550 50  0001 C CNN
 F 3 "~" H 4800 2550 50  0001 C CNN
-F 4 "RC0603JR-07120RL" H 4800 2550 50  0001 C CNN "Partnumber"
+F 4 "180 ohm resistor" H 4800 2550 50  0001 C CNN "Partnumber"
 	1    4800 2550
 	1    0    0    -1
@@
 F 2 "Resistor_SMD:R_0603_1608Metric" V 5480 2550 50  0001 C CNN
 F 3 "~" H 5550 2550 50  0001 C CNN
-F 4 "RC0603JR-07120RL" H 5550 2550 50  0001 C CNN "Partnumber"
+F 4 "180 ohm resistor" H 5550 2550 50  0001 C CNN "Partnumber"
 	1    5550 2550
 	1    0    0    -1
@@
 F 2 "Resistor_SMD:R_0603_1608Metric" V 4330 4500 50  0001 C CNN
 F 3 "~" H 4400 4500 50  0001 C CNN
-F 4 "RC0603JR-07120RL" H 4400 4500 50  0001 C CNN "Partnumber"
+F 4 "180 ohm resistor" H 4400 4500 50  0001 C CNN "Partnumber"
 	1    4400 4500
 	1    0    0    -1
@@
 F 2 "Resistor_SMD:R_0603_1608Metric" V 8880 4500 50  0001 C CNN
 F 3 "~" H 8950 4500 50  0001 C CNN
-F 4 "RC0603JR-07120RL" H 8950 4500 50  0001 C CNN "Partnumber"
+F 4 "180 ohm resistor" H 8950 4500 50  0001 C CNN "Partnumber"
 	1    8950 4500
 	1    0    0    -1

Commit message: *E updates
Parts:
- removed SW1: Off On, iGrillRPiSSRCtl-rev-sE:SW_OS202011MS2QS1, symbol Switch:SW_DPDT_x2
- added SW1: SW_SPDT, Button_Switch_THT:SW_Slide_1P2T_CK_OS102011MS2Q, symbol Switch:SW_SPDT
- R1, R11, R12, R14, R16, R3, R5, R7, R9: value 180Ω -> 1kΩ
Connections:
- wire segments 179 -> 182
Changed lines of the file:
@@
 Sheet 1 1
 Title "iGrill Smoker SSR Control Board"
-Date "2019-08-02"
+Date "2019-08-03"
 Rev "*E"
 Comp "Redbud Farms"
@@
 P 850 1550
 F 0 "R1" V 950 1550 50  0000 C CNN
-F 1 "180Ω" V 850 1550 50  0000 C CNN
+F 1 "1kΩ" V 850 1550 50  0000 C CNN
 F 2 "Resistor_SMD:R_0603_1608Metric" V 780 1550 50  0001 C CNN
 F 3 "~" H 850 1550 50  0001 C CNN
@@
 P 1600 1550
 F 0 "R3" V 1700 1550 50  0000 C CNN
-F 1 "180Ω" V 1600 1550 50  0000 C CNN
+F 1 "1kΩ" V 1600 1550 50  0000 C CNN
 F 2 "Resistor_SMD:R_0603_1608Metric" V 1530 1550 50  0001 C CNN
 F 3 "~" H 1600 1550 50  0001 C CNN
@@
 	0    1    1    0
 $EndComp
-$Comp
-L Switch:SW_DPDT_x2 SW1
-U 2 1 5D19CE23
-P 8350 4350
-F 0 "SW1" H 8350 4635 50  0000 C CNN
-F 1 "Off    On" H 8350 4544 50  0000 C CNN
-F 2 "iGrillRPiSSRCtl-rev-sE:SW_OS202011MS2QS1" H 8350 4350 50  0001 C CNN
-F 3 "~" H 8350 4350 50  0001 C CNN
-F 4 "JS202011SCQN" H 8350 4350 50  0001 C CNN "Partnumber"
-	2    8350 4350
-	-1   0    0    -1
-$EndComp
 Wire Wire Line
 	9300 4350 9350 4350
@@
 $EndComp
 $Comp
-L Switch:SW_DPDT_x2 SW1
-U 1 1 5D23056E
-P 3850 4250
-F 0 "SW1" H 3850 4535 50  0000 C CNN
-F 1 "Off    On" H 3850 4444 50  0000 C CNN
-F 2 "iGrillRPiSSRCtl-rev-sE:SW_OS202011MS2QS1" H 3850 4250 50  0001 C CNN
-F 3 "~" H 3850 4250 50  0001 C CNN
-F 4 "JS202011SCQN" H 3850 4250 50  0001 C CNN "Partnumber"
-	1    3850 4250
-	-1   0    0    -1
-$EndComp
-$Comp
 L power:+5V #PWR06
 U 1 1 5D252AFC
@@
 	3500 4350 3500 4400
 Wire Wire Line
-	3650 4150 3500 4150
-Wire Wire Line
 	3500 4150 3500 4100
 Wire Wire Line
 	3500 4150 3200 4150
-Connection ~ 3500 4150
 Wire Wire Line
 	6550 4250 8150 4250
@@
 P 2350 1550
 F 0 "R5" V 2450 1550 50  0000 C CNN
-F 1 "180Ω" V 2350 1550 50  0000 C CNN
+F 1 "1kΩ" V 2350 1550 50  0000 C CNN
 F 2 "Resistor_SMD:R_0603_1608Metric" V 2280 1550 50  0001 C CNN
 F 3 "~" H 2350 1550 50  0001 C CNN
@@
 P 3100 1550
 F 0 "R7" V 3200 1550 50  0000 C CNN
-F 1 "180Ω" V 3100 1550 50  0000 C CNN
+F 1 "1kΩ" V 3100 1550 50  0000 C CNN
 F 2 "Resistor_SMD:R_0603_1608Metric" V 3030 1550 50  0001 C CNN
 F 3 "~" H 3100 1550 50  0001 C CNN
@@
 P 3850 1550
 F 0 "R9" V 3950 1550 50  0000 C CNN
-F 1 "180Ω" V 3850 1550 50  0000 C CNN
+F 1 "1kΩ" V 3850 1550 50  0000 C CNN
 F 2 "Resistor_SMD:R_0603_1608Metric" V 3780 1550 50  0001 C CNN
 F 3 "~" H 3850 1550 50  0001 C CNN
@@
 P 4600 1550
 F 0 "R12" V 4700 1550 50  0000 C CNN
-F 1 "180Ω" V 4600 1550 50  0000 C CNN
+F 1 "1kΩ" V 4600 1550 50  0000 C CNN
 F 2 "Resistor_SMD:R_0603_1608Metric" V 4530 1550 50  0001 C CNN
 F 3 "~" H 4600 1550 50  0001 C CNN
@@
 P 5350 1550
 F 0 "R14" V 5450 1550 50  0000 C CNN
-F 1 "180Ω" V 5350 1550 50  0000 C CNN
+F 1 "1kΩ" V 5350 1550 50  0000 C CNN
 F 2 "Resistor_SMD:R_0603_1608Metric" V 5280 1550 50  0001 C CNN
 F 3 "~" H 5350 1550 50  0001 C CNN
@@
 	6650 2950 6650 3050
 Wire Wire Line
-	8550 4350 8950 4350
+	8550 4350 8700 4350
 Wire Wire Line
 	3650 4950 3200 4950
@@
 P 4400 4500
 F 0 "R11" V 4500 4500 50  0000 C CNN
-F 1 "180Ω" V 4400 4500 50  0000 C CNN
+F 1 "1kΩ" V 4400 4500 50  0000 C CNN
 F 2 "Resistor_SMD:R_0603_1608Metric" V 4330 4500 50  0001 C CNN
 F 3 "~" H 4400 4500 50  0001 C CNN
@@
 P 8950 4500
 F 0 "R16" V 9050 4500 50  0000 C CNN
-F 1 "180Ω" V 8950 4500 50  0000 C CNN
+F 1 "1kΩ" V 8950 4500 50  0000 C CNN
 F 2 "Resistor_SMD:R_0603_1608Metric" V 8880 4500 50  0001 C CNN
 F 3 "~" H 8950 4500 50  0001 C CNN
@@
 	1    0    0    -1
 $EndComp
-Wire Wire Line
-	8000 3950 8000 4450
-Wire Wire Line
-	8000 4450 8150 4450
-Wire Wire Line
-	6650 3950 8000 3950
+$Comp
+L Switch:SW_SPDT SW1
+U 1 1 5D54B71B
+P 8350 4350
+F 0 "SW1" H 8350 4635 50  0001 C CNN
+F 1 "SW_SPDT" H 8350 4635 50  0000 C CNN
+F 2 "Button_Switch_THT:SW_Slide_1P2T_CK_OS102011MS2Q" H 8350 4350 50  0001 C CNN
+F 3 "~" H 8350 4350 50  0001 C CNN
+F 4 "Off   On" V 8350 4350 50  0000 C CNN "Text"
+	1    8350 4350
+	-1   0    0    -1
+$EndComp
+Wire Wire Line
+	4050 4250 4050 5200
+Wire Wire Line
+	4050 5200 8700 5200
+Wire Wire Line
+	8700 5200 8700 4350
+Connection ~ 8700 4350
+Wire Wire Line
+	8700 4350 8950 4350
+Wire Wire Line
+	8150 4450 8050 4450
+Wire Wire Line
+	8050 4450 8050 3950
+Wire Wire Line
+	6650 3950 8050 3950
 $EndSCHEMATC

Commit message: Fixing pulldown resistors
Parts:
- added R18, R19, R20, R21, R22, R23, R24, R25, R26: 10kΩ, Resistor_SMD:R_0603_1608Metric, symbol Device:R
- R1, R12, R14, R3, R5, R7, R9: value 1kΩ -> 180Ω
- R10, R13, R15, R2, R4, R6, R8: value 180Ω -> 1kΩ
Connections:
- wire segments 182 -> 211

Commit message: Fixed References
Parts:
- R10, R11, R13, R15, R16, R2, R4, R6, R8: Partnumber 180 ohm resistor -> 1k ohm resistor
- R18, R19, R20, R21, R22, R23, R24, R25, R26: Partnumber 180 ohm resistor -> 10k ohm resistor
Changed lines of the file:
@@
 Sheet 1 1
 Title "iGrill Smoker SSR Control Board"
-Date "2019-08-03"
+Date "2019-08-05"
 Rev "*E"
 Comp "Redbud Farms"
@@
 F 2 "Resistor_SMD:R_0603_1608Metric" V 980 2550 50  0001 C CNN
 F 3 "~" H 1050 2550 50  0001 C CNN
-F 4 "180 ohm resistor" H 1050 2550 50  0001 C CNN "Partnumber"
+F 4 "1k ohm resistor" H 1050 2550 50  0001 C CNN "Partnumber"
 	1    1050 2550
 	1    0    0    -1
@@
 F 2 "Resistor_SMD:R_0603_1608Metric" V 1730 2550 50  0001 C CNN
 F 3 "~" H 1800 2550 50  0001 C CNN
-F 4 "180 ohm resistor" H 1800 2550 50  0001 C CNN "Partnumber"
+F 4 "1k ohm resistor" H 1800 2550 50  0001 C CNN "Partnumber"
 	1    1800 2550
 	1    0    0    -1
@@
 F 2 "Resistor_SMD:R_0603_1608Metric" V 2480 2550 50  0001 C CNN
 F 3 "~" H 2550 2550 50  0001 C CNN
-F 4 "180 ohm resistor" H 2550 2550 50  0001 C CNN "Partnumber"
+F 4 "1k ohm resistor" H 2550 2550 50  0001 C CNN "Partnumber"
 	1    2550 2550
 	1    0    0    -1
@@
 F 2 "Resistor_SMD:R_0603_1608Metric" V 3230 2550 50  0001 C CNN
 F 3 "~" H 3300 2550 50  0001 C CNN
-F 4 "180 ohm resistor" H 3300 2550 50  0001 C CNN "Partnumber"
+F 4 "1k ohm resistor" H 3300 2550 50  0001 C CNN "Partnumber"
 	1    3300 2550
 	1    0    0    -1
@@
 F 2 "Resistor_SMD:R_0603_1608Metric" V 3980 2550 50  0001 C CNN
 F 3 "~" H 4050 2550 50  0001 C CNN
-F 4 "180 ohm resistor" H 4050 2550 50  0001 C CNN "Partnumber"
+F 4 "1k ohm resistor" H 4050 2550 50  0001 C CNN "Partnumber"
 	1    4050 2550
 	1    0    0    -1
@@
 F 2 "Resistor_SMD:R_0603_1608Metric" V 4730 2550 50  0001 C CNN
 F 3 "~" H 4800 2550 50  0001 C CNN
-F 4 "180 ohm resistor" H 4800 2550 50  0001 C CNN "Partnumber"
+F 4 "1k ohm resistor" H 4800 2550 50  0001 C CNN "Partnumber"
 	1    4800 2550
 	1    0    0    -1
@@
 F 2 "Resistor_SMD:R_0603_1608Metric" V 5480 2550 50  0001 C CNN
 F 3 "~" H 5550 2550 50  0001 C CNN
-F 4 "180 ohm resistor" H 5550 2550 50  0001 C CNN "Partnumber"
+F 4 "1k ohm resistor" H 5550 2550 50  0001 C CNN "Partnumber"
 	1    5550 2550
 	1    0    0    -1
@@
 F 2 "Resistor_SMD:R_0603_1608Metric" V 4330 4500 50  0001 C CNN
 F 3 "~" H 4400 4500 50  0001 C CNN
-F 4 "180 ohm resistor" H 4400 4500 50  0001 C CNN "Partnumber"
+F 4 "1k ohm resistor" H 4400 4500 50  0001 C CNN "Partnumber"
 	1    4400 4500
 	1    0    0    -1
@@
 F 2 "Resistor_SMD:R_0603_1608Metric" V 8880 4500 50  0001 C CNN
 F 3 "~" H 8950 4500 50  0001 C CNN
-F 4 "180 ohm resistor" H 8950 4500 50  0001 C CNN "Partnumber"
+F 4 "1k ohm resistor" H 8950 4500 50  0001 C CNN "Partnumber"
 	1    8950 4500
 	1    0    0    -1
@@
 F 2 "Resistor_SMD:R_0603_1608Metric" V 830 3000 50  0001 C CNN
 F 3 "~" H 900 3000 50  0001 C CNN
-F 4 "180 ohm resistor" H 900 3000 50  0001 C CNN "Partnumber"
+F 4 "10k ohm resistor" H 900 3000 50  0001 C CNN "Partnumber"
 	1    900  3000
 	0    1    1    0
@@
 F 2 "Resistor_SMD:R_0603_1608Metric" V 1580 3100 50  0001 C CNN
 F 3 "~" H 1650 3100 50  0001 C CNN
-F 4 "180 ohm resistor" H 1650 3100 50  0001 C CNN "Partnumber"
+F 4 "10k ohm resistor" H 1650 3100 50  0001 C CNN "Partnumber"
 	1    1650 3100
 	0    1    1    0
@@
 F 2 "Resistor_SMD:R_0603_1608Metric" V 2330 3200 50  0001 C CNN
 F 3 "~" H 2400 3200 50  0001 C CNN
-F 4 "180 ohm resistor" H 2400 3200 50  0001 C CNN "Partnumber"
+F 4 "10k ohm resistor" H 2400 3200 50  0001 C CNN "Partnumber"
 	1    2400 3200
 	0    1    1    0
@@
 F 2 "Resistor_SMD:R_0603_1608Metric" V 3080 2850 50  0001 C CNN
 F 3 "~" H 3150 2850 50  0001 C CNN
-F 4 "180 ohm resistor" H 3150 2850 50  0001 C CNN "Partnumber"
+F 4 "10k ohm resistor" H 3150 2850 50  0001 C CNN "Partnumber"
 	1    3150 2850
 	0    1    1    0
@@
 F 2 "Resistor_SMD:R_0603_1608Metric" V 3830 2950 50  0001 C CNN
 F 3 "~" H 3900 2950 50  0001 C CNN
-F 4 "180 ohm resistor" H 3900 2950 50  0001 C CNN "Partnumber"
+F 4 "10k ohm resistor" H 3900 2950 50  0001 C CNN "Partnumber"
 	1    3900 2950
 	0    1    1    0
@@
 F 2 "Resistor_SMD:R_0603_1608Metric" V 4580 2800 50  0001 C CNN
 F 3 "~" H 4650 2800 50  0001 C CNN
-F 4 "180 ohm resistor" H 4650 2800 50  0001 C CNN "Partnumber"
+F 4 "10k ohm resistor" H 4650 2800 50  0001 C CNN "Partnumber"
 	1    4650 2800
 	0    1    1    0
@@
 F 2 "Resistor_SMD:R_0603_1608Metric" V 5130 2600 50  0001 C CNN
 F 3 "~" H 5200 2600 50  0001 C CNN
-F 4 "180 ohm resistor" H 5200 2600 50  0001 C CNN "Partnumber"
+F 4 "10k ohm resistor" H 5200 2600 50  0001 C CNN "Partnumber"
 	1    5200 2600
 	-1   0    0    1
@@
 F 2 "Resistor_SMD:R_0603_1608Metric" V 8430 5350 50  0001 C CNN
 F 3 "~" H 8500 5350 50  0001 C CNN
-F 4 "180 ohm resistor" H 8500 5350 50  0001 C CNN "Partnumber"
+F 4 "10k ohm resistor" H 8500 5350 50  0001 C CNN "Partnumber"
 	1    8500 5350
 	-1   0    0    1
@@
 F 2 "Resistor_SMD:R_0603_1608Metric" V 3680 4600 50  0001 C CNN
 F 3 "~" H 3750 4600 50  0001 C CNN
-F 4 "180 ohm resistor" H 3750 4600 50  0001 C CNN "Partnumber"
+F 4 "10k ohm resistor" H 3750 4600 50  0001 C CNN "Partnumber"
 	1    3750 4600
 	0    -1   -1   0
