File: kicad/iGrillRPiSSRCtl-revsE/iGrillRPiSSRCtl-rev-sE.kicad_pcb (KiCad board)
At the start: 2 copper layers, 65 x 56 mm, 65 parts, among them J1 Screw_Terminal_01x02, P1 Conn_02x20_Odd_Even, Q1 MMBT3904LT1G, Q2 MMBT3904LT1G, Q3 MMBT3904LT1G, Q4 MMBT3904LT1G, Q5 MMBT3904LT1G, Q6 MMBT3904LT1G, Q7 MMBT3904LT1G, Q8 MMBT3904LT1G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

Commit message: *E updates before production
Parts:
- BZ1: footprint iGrillRPiSSRCtl-rev-sE:Buzzer_KELIKING_KLJ-1230-smd -> Buzzer_Beeper:Buzzer_TDK_PS1240P02BT_D12.2mm_H6.5mm
- J1: footprint TerminalBlock:TerminalBlock_bornier-2_P5.08mm -> TerminalBlock_Phoenix:TerminalBlock_Phoenix_MKDS-1,5-2-5.08_1x02_P5.08mm_Horizontal
- R17: moved to B.Cu
- moved R17 6.64 mm to (73.9, 41.7), turned to 0 degrees
- moved BZ1 4.32 mm to (71.0, 44.1), turned to 0 degrees
- moved J1 0.08 mm to (79.1, 33.7)
Routing:
- net +5V: track 27.5 -> 30.8 mm
- net Net-(BZ1-Pad2): track 8.82 -> 7.45 mm, vias 1 -> 0
